File: HW/PowerBoard_v1/power_v1.kicad_pcb (KiCad board)
At the start: 4 copper layers, 81.3 x 81 mm, 186 parts, among them J1 Conn_01x03, J10 Conn_01x02, J11 Conn_01x02, J12 Conn_01x03, J14 Conn_01x02, J15 Conn_01x02, J16 Conn_01x02, J17 Conn_01x03, J18 Conn_01x04, J19 Conn_01x02, J2 Conn_01x03, J20 Conn_01x05, J21 Conn_01x05, J22 Conn_01x03, J3 JTAG_header, J4 Conn_01x03, J5 USB_B_Micro, J6 Conn_01x04, J7 Conn_01x06, J8 Conn_01x02, J9 Conn_01x06, Q1 PMOS 30V, Q10 NMOS 20V, Q3 NMOS 30V, Q4 PMOS 30V, Q5 PMOS 30V, Q6 PMOS 30V, Q7 NMOS 30V, Q8 PMOS 20V, Q9 NMOS 20V, SW1 ~{RESET}, SW2 223AMVAAR, U1 MCP9700AT-ETT, U10 MCP1754, U11 MCP9700AT-ETT, U12 PCA9745B, U13 PCA9745B, U14 DSM7TAxx1xxT, U15 DSM7TAxx1xxT, U16 DSM7TAxx1xxT, U17 DSM7TAxx1xxT, U2 LPC1549JBD100, U3 LTC4412, U4 R-78E12-0.5, U5 LM2940x-10, U6 R-78AA3.3-0.5SMD, U7 WE-TVS_82400102, U8 AZ1117-3.3, U9 ISO1042DW, Y1 12MHz

Commit message: small layout changes
Parts:
- removed C29: 4.7uF, Capacitor_SMD:C_0603_1608Metric_Pad1.08x0.95mm_HandSolder
- removed C30, C31, C32, C39, C40, C41, C42: 0.1uF, Capacitor_SMD:C_0603_1608Metric_Pad1.08x0.95mm_HandSolder
- removed C33, C34: 1uF, Capacitor_SMD:C_0603_1608Metric_Pad1.08x0.95mm_HandSolder
- removed C35, C36, C37, C38: 10uF, Capacitor_SMD:C_0805_2012Metric_Pad1.18x1.45mm_HandSolder
- removed D10: PESD1CAN, Package_TO_SOT_SMD:SOT-23
- removed D11: RED, LED_SMD:LED_0603_1608Metric_Pad1.05x0.95mm_HandSolder
- removed D4: LOCAL, LED_SMD:LED_0603_1608Metric_Pad1.05x0.95mm_HandSolder
- removed D6, D8: 30V, Diode_SMD:D_SOD-323_HandSoldering
- removed D7: 5V6, Diode_SMD:D_SOD-123F
- removed D9: 3V6, Diode_SMD:D_SOD-123F
- removed F2: 1A, Fuse:Fuse_0603_1608Metric_Pad1.05x0.95mm_HandSolder
- removed F3: 750mA, Fuse:Fuse_0603_1608Metric_Pad1.05x0.95mm_HandSolder
- removed F4: 0.5A, Fuse:Fuse_0603_1608Metric_Pad1.05x0.95mm_HandSolder
- removed F5, F6: 0.2A, Fuse:Fuse_1206_3216Metric_Pad1.42x1.75mm_HandSolder
- removed H1, H2, H3, H4: MountingHole, MountingHole:MountingHole_2.5mm
- removed J10, J11, J14, J15, J16, J19, J8: Conn_01x02, Connector_Molex:Molex_PicoBlade_53398-0271_1x02-1MP_P1.25mm_Vertical
- removed J12, J17, J2, J22: Conn_01x03, Connector_Molex:Molex_PicoBlade_53398-0371_1x03-1MP_P1.25mm_Vertical
- removed J18, J6: Conn_01x04, Connector_Molex:Molex_PicoBlade_53398-0471_1x04-1MP_P1.25mm_Vertical
- removed J20, J21: Conn_01x05, Connector_Molex:Molex_PicoBlade_53398-0571_1x05-1MP_P1.25mm_Vertical
- removed J7, J9: Conn_01x06, Connector_Molex:Molex_PicoBlade_53398-0671_1x06-1MP_P1.25mm_Vertical
- removed MK1: ISC Logo, layout:ISC_Circles_5mm_x_4mm
- removed MK2: BAC Logo, layout:BAC_Square_Logo_5mm
- removed MK3: Block I, layout:BLOCK_I_5mm_x_3.4mm
- removed MK4: ISC Logo, layout:ISC_BLogo
- removed MK5: BAC Logo, layout:BAC_Full_Logo_41.1mm_x_12.1mm
- removed Q10, Q9: NMOS 20V, Package_TO_SOT_SMD:SOT-23_Handsoldering
- removed Q3, Q7: NMOS 30V, Package_TO_SOT_SMD:SOT-23_Handsoldering
- removed Q4, Q5, Q6: PMOS 30V, Package_TO_SOT_SMD:SOT-23_Handsoldering
- removed Q8: PMOS 20V, Package_TO_SOT_SMD:SOT-23_Handsoldering
- removed R12: 0, Resistor_SMD:R_0603_1608Metric_Pad0.98x0.95mm_HandSolder
- removed R13, R14, R15: 10K, Resistor_SMD:R_0603_1608Metric_Pad0.98x0.95mm_HandSolder
- removed R16, R20, R22, R36, R37, R38, R39, R40, R42, R43, R44, R45, R46, R47, R48, R51: 1k, Resistor_SMD:R_0603_1608Metric_Pad0.98x0.95mm_HandSolder
- removed R17, R18, R19, R25, R26, R34, R35, R41: 10k, Resistor_SMD:R_0603_1608Metric_Pad0.98x0.95mm_HandSolder
- removed R21: 470k, Resistor_SMD:R_0603_1608Metric_Pad0.98x0.95mm_HandSolder
- removed R23, R30, R32, R33: 100k, Resistor_SMD:R_0603_1608Metric_Pad0.98x0.95mm_HandSolder
- removed R24: 24.9k, Resistor_SMD:R_0603_1608Metric_Pad0.98x0.95mm_HandSolder
- removed R27: 22, Resistor_SMD:R_2512_6332Metric_Pad1.40x3.35mm_HandSolder
- removed R28: DNP, Resistor_SMD:R_0603_1608Metric_Pad0.98x0.95mm_HandSolder
- removed R29: 6.8, Resistor_SMD:R_2512_6332Metric_Pad1.40x3.35mm_HandSolder
- removed R31: 7.5k, Resistor_SMD:R_0603_1608Metric_Pad0.98x0.95mm_HandSolder
- removed R49: 1M, Resistor_SMD:R_0603_1608Metric_Pad0.98x0.95mm_HandSolder
- removed R50: 120, Resistor_SMD:R_0603_1608Metric_Pad0.98x0.95mm_HandSolder
- removed R52, R53: 2k, Resistor_SMD:R_0603_1608Metric_Pad0.98x0.95mm_HandSolder
- removed S1: CL-SB-22A, layout:DPDT_NIDEC_6_pin_SMD_1.6_x_1.2_pads
- removed SW1: ~{RESET}, layout:Button_223AM
- removed SW2: 223AMVAAR, layout:Button_223AM
- removed TP14: MOSI, TestPoint:TestPoint_THTPad_D1.0mm_Drill0.5mm
- removed TP15: CLK, TestPoint:TestPoint_THTPad_D1.0mm_Drill0.5mm
- removed TP16: +3v3, TestPoint:TestPoint_THTPad_D1.0mm_Drill0.5mm
- removed U10: MCP1754, Package_TO_SOT_SMD:SOT-23
- removed U11: MCP9700AT-ETT, Package_TO_SOT_SMD:SOT-23
- removed U12, U13: PCA9745B, layout:PCA9745B
- removed U14, U15, U16, U17: DSM7TAxx1xxT, layout:DSM7TA28101T-Front-HandSolder
- removed U9: ISO1042DW, layout:SOIC-8_5.85x7.4mm_P1.27mm
- removed Y1: 12MHz, Crystal:Crystal_SMD_3225-4Pin_3.2x2.5mm_HandSoldering
- added JP1: SolderJumper_2_Open, Resistor_SMD:R_0603_1608Metric_Pad0.98x0.95mm_HandSolder, F.Cu at (211.0, 39.1)
- added L1: 1.2 μH, Inductor_SMD:L_Wuerth_HCM-1050, F.Cu at (202.8, 27.2)
- added L2: 1.2 μH, Inductor_SMD:L_Wuerth_HCM-1050, F.Cu at (202.8, 35.9)
- added L3: 22uH, Inductor_SMD:L_0603_1608Metric_Pad1.05x0.95mm_HandSolder, F.Cu at (252.5, 63.8)
- added Q2: IXTT220N20X4HV, Package_TO_SOT_SMD:TO-268-2, F.Cu at (173.5, 80.4)
- C1: value 0.16uF -> 10uF; moved to F.Cu
- C10: value 0.01uF -> 100nF
- C11: value 0.01uF -> 100nF; moved to F.Cu
- C12, C13: value 10uF -> 1uF; footprint Capacitor_SMD:C_0805_2012Metric_Pad1.18x1.45mm_HandSolder -> Capacitor_SMD:C_0603_1608Metric_Pad1.08x0.95mm_HandSolder
- C15: value 10uF -> 100nF; footprint Capacitor_SMD:C_0805_2012Metric_Pad1.18x1.45mm_HandSolder -> Capacitor_SMD:C_0603_1608Metric_Pad1.08x0.95mm_HandSolder; moved to F.Cu
- C16: value 0.1uF -> 100nF
- C17: value 22uF -> 1uF; footprint Capacitor_SMD:C_0805_2012Metric_Pad1.18x1.45mm_HandSolder -> Capacitor_SMD:C_0603_1608Metric_Pad1.08x0.95mm_HandSolder
- C18, C19: value 0.47F -> 1uF; footprint layout:CP_Radial_D16.5mm_P5.08mm -> Capacitor_SMD:C_0603_1608Metric_Pad1.08x0.95mm_HandSolder
- C2: value 0.16uF -> 1nF
- C20: value 10uF -> 100nF
- C21: value 1uF -> 100nF
- C22: value 10uF -> 100nF; footprint Capacitor_SMD:C_0805_2012Metric_Pad1.18x1.45mm_HandSolder -> Capacitor_SMD:C_0603_1608Metric_Pad1.08x0.95mm_HandSolder
- C23: value 22uF -> 100nF
- C24, C4: value 0.1uF -> 1uF
- C25, C3: value 0.1uF -> 1uF; moved to F.Cu
- C26: value 0.1uF -> 10uF; moved to F.Cu
- C27: value 0.1uF -> 2.2nF
- C28: value 0.1uF -> 1nF; moved to B.Cu
- C5, C6: value 22pF -> 1uF
- C7, C8: value 0.1uF -> 470uF; footprint Capacitor_SMD:C_0603_1608Metric_Pad1.08x0.95mm_HandSolder -> Capacitor_THT:C_Radial_D18.0mm_H35.5mm_P7.50mm
- C9: value 10uF -> 0.1uF
- D1: value CONNX -> Blue
- D2: value CAN_RX -> 0.83V; footprint LED_SMD:LED_0603_1608Metric_Pad1.05x0.95mm_HandSolder -> Package_TO_SOT_SMD:TO-252-2
- D3: value CAN_TX -> 0.83V; footprint LED_SMD:LED_0603_1608Metric_Pad1.05x0.95mm_HandSolder -> Package_TO_SOT_SMD:TO-252-2
- J1: value Conn_01x03 -> Inputs; footprint Connector_Molex:Molex_PicoBlade_53398-0371_1x03-1MP_P1.25mm_Vertical -> Connector_Molex:Molex_Micro-Fit_3.0_43650-0400_1x04_P3.00mm_Horizontal
- J3: value JTAG_header -> Vin Solar; footprint layout:IDC-Header_2x05_Pitch1.27mm_Straight -> layout:Anderson_Powerpole_45A_1x2_Horizontal_Bottom
- J4: value Conn_01x03 -> Vout Battery; footprint Connector_Molex:Molex_PicoBlade_53398-0371_1x03-1MP_P1.25mm_Vertical -> layout:Anderson_Powerpole_45A_1x2_Horizontal_Bottom
- J5: value USB_B_Micro -> Sensors; footprint Connector_USB:USB_Micro-B_Molex_47346-0001 -> Connector_Molex:Molex_Micro-Fit_3.0_43650-0500_1x05_P3.00mm_Horizontal
- Q1: value PMOS 30V -> IXTT220N20X4HV; footprint Package_TO_SOT_SMD:SOT-23_Handsoldering -> Package_TO_SOT_SMD:TO-268-2; moved to F.Cu
- R1: value 1k -> 10; moved to F.Cu
- R10: value 1k -> 0.75; footprint Resistor_SMD:R_0603_1608Metric_Pad0.98x0.95mm_HandSolder -> Package_TO_SOT_SMD:TO-263-2_TabPin1
- R11: value 10k -> 0.75; footprint Resistor_SMD:R_0603_1608Metric_Pad0.98x0.95mm_HandSolder -> Package_TO_SOT_SMD:TO-263-2_TabPin1
- R2: value 1k -> 0; moved to F.Cu
- R3: value 1k -> 10k; moved to F.Cu
- R4: value 1k -> 500k; moved to F.Cu
- R5: value 10k -> 500k
- R6: value 1k -> 53k
- R7, R8: value 1k -> 500k
- R9: value 1k -> 41.7k
- TP1: value V_IN -> +3V3A; footprint TestPoint:TestPoint_THTPad_D1.0mm_Drill0.5mm -> TestPoint:TestPoint_THTPad_1.0x1.0mm_Drill0.5mm
- TP10: value CAN_L -> ADC V Sol; footprint TestPoint:TestPoint_THTPad_D1.0mm_Drill0.5mm -> TestPoint:TestPoint_THTPad_1.0x1.0mm_Drill0.5mm
- TP11: value GND_CAN -> ADC V Batt; footprint TestPoint:TestPoint_THTPad_D1.0mm_Drill0.5mm -> TestPoint:TestPoint_THTPad_1.0x1.0mm_Drill0.5mm
- TP12: value DAISYCHAIN -> ADC I Sol; footprint TestPoint:TestPoint_THTPad_D1.0mm_Drill0.5mm -> TestPoint:TestPoint_THTPad_1.0x1.0mm_Drill0.5mm
- TP13: value MISO -> ADC I Batt; footprint TestPoint:TestPoint_THTPad_D1.0mm_Drill0.5mm -> TestPoint:TestPoint_THTPad_1.0x1.0mm_Drill0.5mm
- TP2: value +24V -> GNDA; footprint TestPoint:TestPoint_THTPad_D1.0mm_Drill0.5mm -> TestPoint:TestPoint_THTPad_1.0x1.0mm_Drill0.5mm
- TP3: value GND -> 24V; footprint TestPoint:TestPoint_THTPad_D1.0mm_Drill0.5mm -> TestPoint:TestPoint_THTPad_1.0x1.0mm_Drill0.5mm
- TP4: value V_SuperCap -> GND; footprint TestPoint:TestPoint_THTPad_D1.0mm_Drill0.5mm -> TestPoint:TestPoint_THTPad_1.0x1.0mm_Drill0.5mm
- TP5: value ENC SPI CLK -> 3V3; footprint TestPoint:TestPoint_THTPad_D1.0mm_Drill0.5mm -> TestPoint:TestPoint_THTPad_1.0x1.0mm_Drill0.5mm
- TP6: value ENC SPI MISO -> ADC V Sol; footprint TestPoint:TestPoint_THTPad_D1.0mm_Drill0.5mm -> TestPoint:TestPoint_THTPad_1.0x1.0mm_Drill0.5mm
- TP7: value GND -> ADC V Batt; footprint TestPoint:TestPoint_THTPad_D1.0mm_Drill0.5mm -> TestPoint:TestPoint_THTPad_1.0x1.0mm_Drill0.5mm
- TP8: value +5V_CAN -> ADC I Sol; footprint TestPoint:TestPoint_THTPad_D1.0mm_Drill0.5mm -> TestPoint:TestPoint_THTPad_1.0x1.0mm_Drill0.5mm
- TP9: value CAN_H -> ADC I Batt; footprint TestPoint:TestPoint_THTPad_D1.0mm_Drill0.5mm -> TestPoint:TestPoint_THTPad_1.0x1.0mm_Drill0.5mm
- U1: value MCP9700AT-ETT -> RO-2412S; footprint Package_TO_SOT_SMD:SOT-23 -> Converter_DCDC:Converter_DCDC_RECOM_R-78S-0.1_THT
- U2: value LPC1549JBD100 -> STGAP2SMTR; footprint Package_QFP:LQFP-100_14x14mm_P0.5mm -> Package_SO:SOIC-8_3.9x4.9mm_P1.27mm
- U3: value LTC4412 -> MCP9700AT-ETT; footprint Package_TO_SOT_SMD:SOT-23-6_Handsoldering -> Package_TO_SOT_SMD:SOT-23
- U4: value R-78E12-0.5 -> PAMC1350DWVR; footprint Converter_DCDC:Converter_DCDC_RECOM_R-78E-0.5_THT -> layout:U_PAMC1350DWVR_TEX
- U5: value LM2940x-10 -> PAMC1350DWVR; footprint Package_TO_SOT_SMD:SOT-223-3_TabPin2 -> layout:U_PAMC1350DWVR_TEX
- U6: value R-78AA3.3-0.5SMD -> PAMC1350DWVR; footprint layout:Converter_DCDC_RECOM_R-78AA_SMD -> layout:U_PAMC1350DWVR_TEX
- U7: value WE-TVS_82400102 -> PAMC1350DWVR; footprint Package_TO_SOT_SMD:SOT-23-6_Handsoldering -> layout:U_PAMC1350DWVR_TEX
- U8: value AZ1117-3.3 -> 3v3 ISO DC/DC; footprint Package_TO_SOT_SMD:SOT-223-3_TabPin2 -> Converter_DCDC:Converter_DCDC_RECOM_R-78S-0.1_THT
- moved TP11 168.3 mm to (266.7, 49.0)
- moved TP8 167.2 mm to (263.6, 52.1)
- moved TP9 158.5 mm to (263.6, 55.1)
- moved R4 156.8 mm to (256.9, 48.8), turned to 0 degrees
- moved TP10 155.4 mm to (263.6, 58.2)
- moved C25 154.1 mm to (252.5, 53.8), turned to 0 degrees
- moved TP6 151.3 mm to (260.6, 58.2)
- moved R10 150.5 mm to (250.5, 29.0), turned to 0 degrees
- moved R9 150.3 mm to (256.9, 61.3), turned to 0 degrees
- moved R8 150.2 mm to (256.9, 58.8), turned to 0 degrees
- moved R7 150.1 mm to (256.9, 56.3), turned to 0 degrees
- moved R6 150.0 mm to (256.9, 53.8), turned to 0 degrees
- moved R11 149.9 mm to (250.5, 41.3), turned to 0 degrees
- moved TP5 149.6 mm to (260.6, 55.1)
- moved R5 149.4 mm to (256.9, 51.3), turned to 0 degrees
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Connections:
- C1 pad 1: /USB_D- -> +24V
- C11 pad 1: +3V3 -> +3.3VA
- C11 pad 2: GND -> Earth
- C12 pad 1: /Wheel_v8.1_Power/V_IN -> +3V3
- C13 pad 1: Net-(Q4-D) -> +3.3VA
- C13 pad 2: GND -> Earth
- C14 pad 1: /Wheel_v8.1_Power/V_IN -> +3.3VA
- C14 pad 2: GND -> Earth
- C15 pad 1: Net-(U4-OUT) -> +3.3VA
- C15 pad 2: GND -> Earth
- C17 pad 1: Net-(U5-OUT) -> +3V3
- C18 pad 1: /Wheel_v8.1_Power/V_SuperCap -> +3.3VA
- C18 pad 2: Net-(C18-Pad2) -> Earth
- C19 pad 1: Net-(C18-Pad2) -> +3.3VA
- C19 pad 2: GND -> Earth
- C2 pad 1: /USB_D+ -> +24V
- C20 pad 1: +3V3 -> +3.3VA
- C20 pad 2: GND -> Earth
- C21 pad 1: +3V3 -> +3.3VA
- C21 pad 2: GND -> Earth
- C22 pad 1: /Wheel_v8.1_USB/+5V_USB_FUSED -> +3V3
- C23 pad 1: /Wheel_v8.1_USB/+3V3_USB -> +3V3
- C24 pad 1: /USB_VBUS -> +3V3
- C27 pad 1: +3V3 -> GND
- C27 pad 2: GND -> Earth
- C28 pad 1: /Wheel_v8.1_CAN/CAN_VCC_FUSED -> +3.3VA
- C28 pad 2: /Wheel_v8.1_CAN/GND_CAN -> Net-(U8-+VIN)
- C5 pad 1: GND -> Net-(U1-+VOUT)
- C5 pad 2: /Wheel_v8.1_MCU/XTALIN -> Earth
- C6 pad 1: GND -> Net-(U1-+VOUT)
- C6 pad 2: /Wheel_v8.1_MCU/XTALOUT -> Earth
- C7 pad 1: +3V3 -> /Batt In
- C7 pad 2: GND -> Earth
- C8 pad 1: +3V3 -> /Batt In
- C8 pad 2: GND -> Earth
- D1 pad 1: GND -> Earth
- D2 pad 1: GND -> /DNP Anode
- D2 pad 2: Net-(D2-A) -> /Batt In
- D3 pad 1: GND -> /DNP Anode
- D3 pad 2: Net-(D3-A) -> /Batt In
- J1 pad 1: Net-(J1-Pin_1) -> GND
- J1 pad 2: GND -> /PWM
- J1 pad 3: Net-(J1-Pin_3) -> +24V
- J3 pad 1: Net-(J3-VCC) -> Earth
- J3 pad 2: /Wheel_v8.1_MCU/TMS -> /Sol In
- J4 pad 1: /Conn_Sense -> /Batt Out
- J4 pad 2: /Wheel_v8.1_Power/V_IN_UNFUSED -> Earth
- J5 pad 1: /Wheel_v8.1_USB/+5V_USB_UNFUSED -> /ADC V Sol
- J5 pad 2: Net-(J5-D-) -> /ADC V Batt
- J5 pad 3: Net-(J5-D+) -> /ADC I Sol
- J5 pad 4: unconnected-(J5-ID-Pad4) -> /ADC I Batt
- J5 pad 5: GND -> /Board Temp
- Q1 pad 1: GND -> /Gate
- Q1 pad 2: Net-(Q1-S) -> /DNP Anode
- Q1 pad 3: +24V -> Earth
- R1 pad 1: /L_SIG -> /Gate
- R1 pad 2: Net-(J1-Pin_1) -> /SW_G+
- R10 pad 1: /USB_D+ -> /Sol In
- R10 pad 2: /Wheel_v8.1_MCU/USB_D+ -> /Sol Out
- R11 pad 1: +3V3 -> /Batt Out
- R11 pad 2: /Wheel_v8.1_MCU/ISP_1 -> /Batt In
- R2 pad 1: /IND_L -> /Gate
- R2 pad 2: Net-(J1-Pin_3) -> /SW_G-
- R3 pad 1: /R_SIG -> /Gate
- R3 pad 2: Net-(J2-Pin_1) -> Net-(D1-A)
- R4 pad 1: /IND_R -> /Sol In
- R4 pad 2: Net-(J2-Pin_3) -> Net-(R4-Pad2)
- R5 pad 1: +3V3 -> Net-(R4-Pad2)
- R5 pad 2: /Wheel_v8.1_MCU/ISP_0 -> /Sensors/V Sense Sol
- R6 pad 1: /Wheel_v8.1_MCU/LED0 -> /Sensors/V Sense Sol
- R6 pad 2: Net-(D1-A) -> Earth
- R7 pad 1: /Wheel_v8.1_MCU/LED1 -> /Batt Out
- R7 pad 2: Net-(D2-A) -> Net-(R7-Pad2)
- R8 pad 1: /Wheel_v8.1_MCU/LED2 -> Net-(R7-Pad2)
- R8 pad 2: Net-(D3-A) -> /Sensors/V Sense Batt
- R9 pad 1: /Wheel_v8.1_MCU/LED3 -> /Sensors/V Sense Batt
- R9 pad 2: Net-(D4-A) -> Earth
- TP1 pad 1: /Wheel_v8.1_Power/V_IN -> +3.3VA
- TP10 pad 1: /Wheel_v8.1_CAN/CAN_L -> /Batt In
- TP11 pad 1: /Wheel_v8.1_CAN/GND_CAN -> /Batt Out
- TP12 pad 1: /Wheel_v8.1_Displays/SDO1 -> /Sol Out
- TP13 pad 1: /MISO_DISP -> /Sol In
- TP2 pad 1: +24V -> Earth
- TP3 pad 1: GND -> +24V
- TP4 pad 1: /Wheel_v8.1_Power/V_SuperCap -> GND
- TP5 pad 1: /SCLK_ENC -> +3V3
- TP6 pad 1: /MISO_ENC -> /ADC V Sol
- TP7 pad 1: GND -> /ADC V Batt
- TP8 pad 1: /Wheel_v8.1_CAN/+5V_CAN -> /ADC I Sol
- TP9 pad 1: /Wheel_v8.1_CAN/CAN_H -> /ADC I Batt
- U1 pad 1: +3V3 -> GND
- U1 pad 2: /Board Temp -> +24V
- U1 pad 3: GND -> Earth
- U2 pad 1: /~{LEDRES} -> +3V3
- U2 pad 2: /Wheel_v8.1_Inputs/BTN1 -> /PWM
- U2 pad 3: /MISO_ENC -> GND
- U2 pad 4: +3V3 -> GND
- U2 pad 5: unconnected-(U2-PIO1_0/ADC0_8_-Pad5) -> Net-(U1-+VOUT)
- U2 pad 6: unconnected-(U2-PIO0_1/ADC0_7/SCT0_OUT4-Pad6) -> /SW_G+
- U2 pad 7: GND -> /SW_G-
- U2 pad 8: unconnected-(U2-PIO0_2/ADC0_6/SCT1_OUT3-Pad8) -> Earth
- U3 pad 1: /Wheel_v8.1_Power/V_SuperCap -> +3V3
- U3 pad 2: GND -> /Board Temp
- U4 pad 1: Net-(Q4-D) -> +3.3VA
- U4 pad 2: GND -> /Sensors/V Sense Sol
- U4 pad 3: Net-(U4-OUT) -> Earth
- U5 pad 1: Net-(U4-OUT) -> +3.3VA
- U5 pad 2: GND -> /Sensors/V Sense Batt
- U5 pad 3: Net-(U5-OUT) -> Earth
- U6 pad 1: +24V -> +3.3VA
- U6 pad 2: +24V -> /Sol In
- U6 pad 3: GND -> /Sol Out
- U6 pad 4: Net-(D6-A) -> Earth
- U6 pad 5: Net-(D6-A) -> GND
- U6 pad 6: Net-(U6-Vadj) -> GND
- U6 pad 7: GND -> /ADC I Sol
- U6 pad 8: GND -> +3V3
- U7 pad 1: /USB_D- -> +3.3VA
- U7 pad 2: GND -> /Batt Out
- U7 pad 3: /USB_D+ -> /Batt In
- U7 pad 4: Net-(J5-D+) -> Earth
- U7 pad 5: /Wheel_v8.1_USB/+5V_USB_FUSED -> GND
- U7 pad 6: Net-(J5-D-) -> GND
- U8 pad 2: /Wheel_v8.1_USB/+3V3_USB -> Net-(U8-+VIN)
- U8 pad 3: /Wheel_v8.1_USB/+5V_USB_FUSED -> Earth
Routing:
- net GND: track 231.7 -> 0.00 mm, vias 71 -> 0
- net +3V3: track 109.5 -> 0.00 mm, vias 33 -> 0
- net /~{RESET}: track 96.3 -> 0.00 mm, vias 1 -> 0
- net /SCLK_Disp: track 96.0 -> 0.00 mm, vias 4 -> 0
- net /MOSI_DISP: track 95.4 -> 0.00 mm, vias 4 -> 0
- net /Wheel_v8.1_Inputs/BTN9: track 84.8 -> 0.00 mm, vias 1 -> 0
- net /MISO_DISP: track 84.0 -> 0.00 mm, vias 4 -> 0
- net /Wheel_v8.1_Inputs/BTN3: track 82.1 -> 0.00 mm, vias 1 -> 0
- net /PTT_SENSE: track 75.7 -> 0.00 mm, vias 1 -> 0
- net /Wheel_v8.1_Inputs/BTN2: track 68.5 -> 0.00 mm, vias 1 -> 0
- net /USB_D-: track 66.3 -> 0.00 mm, vias 4 -> 0
- net /~{LEDRES}: track 65.3 -> 0.00 mm, vias 3 -> 0
- net /L_SIG: track 64.3 -> 0.00 mm, vias 1 -> 0
- net /Wheel_v8.1_MCU/USB_D+: track 61.9 -> 0.00 mm, vias 2 -> 0
- net /IND_L: track 61.0 -> 0.00 mm, vias 1 -> 0
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- removed copper zone on In1.Cu, net +3V3
- removed copper zone on F.Cu, net /MISO_ENC
- removed copper zone on In1.Cu, net /Wheel_v8.1_CAN/+5V_CAN
- removed copper zone on In2.Cu, net /Wheel_v8.1_CAN/GND_CAN
- removed copper zone on F.Cu, net /Wheel_v8.1_Power/V_SuperCap
- removed copper zone on B.Cu, net GND
- removed copper zone on F.Cu, net GND
- removed copper zone on In2.Cu, net GND
Other:
- board outline removed
- board text removed: "+12V"
- board text removed: "+24V"
- board text removed: "+3v3"
- board text removed: "3v3"
- board text removed: "5V_CAN"
- board text removed: ":("
- board text removed: "CAN"
- board text removed: "CAN_GND"
- board text removed: "CC+"
- board text removed: "CC-"
- board text removed: "CC_EN"
- board text removed: "COAST"
- board text removed: "CS"
- board text removed: "DAISYCHAIN"
- board text removed: "DIR_BTN"
- board text removed: "DO"
- board text removed: "DO1"
- board text removed: "Designed by: Alex Chmiel Alex Lymberopoulos Johnathan Vogt"
- board text removed: "ENCODERS"
- board text removed: "FLAG"
- board text removed: "GND"
- board text removed: "GND 3V3 GND"
- board text removed: "H"
- board text removed: "HORN"
- board text removed: "IND_L"
- board text removed: "IND_R"
- board text removed: "L"
- board text removed: "LED CONNECTIONS"
- board text removed: "L_SIG"
- board text removed: "MISO"
- board text removed: "MOSI"
- board text removed: "NC"
- board text removed: "NO"
- board text removed: "OLED"
- board text removed: "PRGM"
- board text removed: "PTT BUTTON"
- board text removed: "PTT OUT"
- board text removed: "R"
- board text removed: "RES"
- board text removed: "RESET"
- board text removed: "R_SIG"
- board text removed: "SCLK"
- board text removed: "SH"
- board text removed: "Sense"
- board text removed: "Serial #"
- board text removed: "TURN SIG"
- board text removed: "UP GND DN"
- board text removed: "V_CAP"
- board text removed: "V_IN"
- board text removed: "Wheel v8.1 10/23"
- board text removed: "not LPC1768 lol"
- board text removed: "~{CS}"
- board text removed: "~{RES}"
- board text removed: "← TERM"

Commit message: need to figure out current sense res fp
Parts:
- removed R10, R11: 0.75, Package_TO_SOT_SMD:TO-263-2_TabPin1
- C28: moved to F.Cu
- moved C28 190.1 mm to (312.9, -12.5), turned to 0 degrees
- moved J3 173.9 mm to (96.7, 179.4), turned to 0 degrees
- moved C1 167.5 mm to (249.1, -26.6), turned to 0 degrees
- moved C2 167.3 mm to (249.1, -24.1), turned to 0 degrees
- moved R6 150.6 mm to (117.2, 110.0), turned to -90 degrees
- moved R5 149.8 mm to (117.2, 105.5), turned to -90 degrees
- moved R4 149.3 mm to (117.2, 101.5), turned to -90 degrees
- moved D3 144.6 mm to (82.7, 82.5), turned to 90 degrees
- moved J4 140.6 mm to (91.7, 6.06), turned to 180 degrees
- moved L2 138.9 mm to (95.7, 124.5), turned to -90 degrees
- moved JP1 137.8 mm to (103.2, 125.0), turned to -90 degrees
- moved U6 135.2 mm to (127.2, 124.0)
- moved L1 134.3 mm to (110.2, 124.5), turned to 90 degrees
- moved D2 134.1 mm to (97.2, 82.5), turned to 90 degrees
- moved U4 132.5 mm to (129.2, 107.0)
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Routing:
- net Earth: track 0.00 -> 19.9 mm, vias 0 -> 2
- net GND: track 0.00 -> 10.2 mm, vias 0 -> 3
- net /Sensors/V Sense Sol: track 0.00 -> 9.31 mm
- net +3V3: track 0.00 -> 8.29 mm
- net +3.3VA: track 0.00 -> 6.82 mm
- net Net-(R4-Pad2): track 0.00 -> 2.18 mm

Commit message: more layout
Parts:
- added R10: 0.75, Package_TO_SOT_SMD:TO-263-2_isolatedback, F.Cu at (95.3, 143.4)
- added R11: 0.75, Package_TO_SOT_SMD:TO-263-2_isolatedback, F.Cu at (101.2, 42.0)
- moved C18 232.5 mm to (120.7, 117.0), turned to 180 degrees
- moved C20 231.4 mm to (120.7, 120.0), turned to 180 degrees
- moved C24 223.9 mm to (140.2, 120.0)
- moved C22 214.9 mm to (140.2, 123.5)
- moved U7 173.3 mm to (129.2, 73.0)
- moved U5 164.8 mm to (129.2, 64.5)
- moved U2 162.0 mm to (129.2, 93.0), turned to 180 degrees
- moved U1 66.5 mm to (133.0, 81.8)
- moved J1 41.5 mm to (153.4, 119.3)
- moved J5 41.5 mm to (153.4, 97.3)
- moved JP1 9.85 mm to (94.2, 129.0)
- moved L1 9.85 mm to (101.2, 128.5)
- moved L2 9.85 mm to (86.7, 128.5)
- moved C7 7.50 mm to (85.0, 63.0), turned to 180 degrees
- moved U6 2.50 mm to (129.2, 125.5)
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Routing:
- net GND: track 10.2 -> 21.4 mm, vias 3 -> 6
- net +3V3: track 8.29 -> 16.6 mm
- net +3.3VA: track 6.82 -> 14.3 mm
- net Earth: track 19.9 -> 22.9 mm
- added copper zone on F.Cu, net +3.3VA
- added copper zone on F.Cu, net +3V3
- added copper zone on B.Cu, net Earth
- added copper zone on B.Cu, net GND
Other:
- copper layers 4 -> 2

Commit message: more changes
Parts:
- C1, C2, C4, C5, C6: moved to B.Cu
- moved U3 250.5 mm to (112.7, 126.0), turned to 180 degrees
- moved C9 246.4 mm to (112.7, 130.0), turned to 180 degrees
- moved L3 222.7 mm to (136.7, 127.0), turned to -90 degrees
- moved R8 220.9 mm to (116.2, 76.5)
- moved R7 220.1 mm to (116.2, 72.0), turned to 180 degrees
- moved C19 204.1 mm to (120.2, 61.0), turned to 180 degrees
- moved C21 203.5 mm to (120.2, 64.5), turned to 180 degrees
- moved C15 202.3 mm to (120.2, 74.0), turned to 180 degrees
- moved C14 202.1 mm to (120.2, 71.0), turned to 180 degrees
- moved C16 196.8 mm to (138.2, 73.5)
- moved C23 196.4 mm to (138.3, 65.0)
- moved C17 194.1 mm to (138.2, 70.5)
- moved C25 192.7 mm to (138.3, 61.5)
- moved D1 167.7 mm to (119.2, 96.5)
- moved C5 166.8 mm to (124.2, 94.0), turned to -90 degrees
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Connections:
- J1 pad 2: /PWM -> +3V3
- J1 pad 4: +3V3 -> /PWM
- J5 pad 1: /ADC V Sol -> /ADC I Batt
- J5 pad 3: /ADC I Sol -> /Board Temp
- J5 pad 4: /ADC I Batt -> /ADC V Sol
- J5 pad 5: /Board Temp -> /ADC I Sol
- R11 pad 1: /Batt Out -> /Batt In
- R11 pad 2: /Batt In -> /Batt Out
- R7 pad 1: /Batt Out -> /Batt In
- TP10 pad 1: /Batt In -> /Batt Out
- TP11 pad 1: /Batt Out -> /Batt In
- U7 pad 2: /Batt Out -> /Batt In
- U7 pad 3: /Batt In -> /Batt Out
Routing:
- net GND: track 21.4 -> 35.8 mm, vias 6 -> 7
- net Earth: track 22.9 -> 29.4 mm
- net +24V: track 0.00 -> 3.00 mm
- net +3.3VA: track 14.3 -> 16.3 mm
Other:
- board text added: "Team #25 Alex Lymberopoulos Alex Chmiel Akhil Pothineni"

Commit message: added changes
Parts:
- moved R9 224.9 mm to (113.7, 83.0), turned to -90 degrees
- moved R7 3.97 mm to (113.7, 75.1), turned to -90 degrees
- moved R8 3.54 mm to (113.7, 79.0), turned to -90 degrees
Changed lines of the file:
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@@
 	(footprint "Resistor_SMD:R_0603_1608Metric_Pad0.98x0.95mm_HandSolder"
 		(layer "F.Cu")
-		(at 116.2 76.5)
+		(at 113.7 79 -90)
 		(descr "Resistor SMD 0603 (1608 Metric), square (rectangular) end terminal, IPC_7351 nominal with elongated pad for handsoldering. (Body size source: IPC-SM-782 page 72, https://www.pcb-3d.com/wordpress/wp-content/uploads/ipc-sm-782a_amendment_1_and_2.pdf), generated with kicad-footprint-generator")
 		(tags "resistor handsolder")
 		(property "Reference" "R8"
-			(at 0 -1.43 0)
+			(at 0 -1.43 90)
 			(layer "F.SilkS")
 			(effects
@@
 		)
 		(property "Value" "500k"
-			(at 0 1.43 0)
+			(at 0 1.43 90)
 			(layer "F.Fab")
 			(effects
@@
 		)
 		(property "Footprint" "Resistor_SMD:R_0603_1608Metric_Pad0.98x0.95mm_HandSolder"
-			(at 0 0 0)
+			(at 0 0 -90)
 			(unlocked yes)
 			(layer "F.Fab")
@@
 		)
 		(property "Datasheet" ""
-			(at 0 0 0)
+			(at 0 0 -90)
 			(unlocked yes)
 			(layer "F.Fab")
@@
 		)
 		(property "Description" "Resistor, US symbol"
-			(at 0 0 0)
+			(at 0 0 -90)
 			(unlocked yes)
 			(layer "F.Fab")
@@
 		(attr smd)
 		(fp_line
-			(start -0.254724 -0.5225)
-			(end 0.254724 -0.5225)
+			(start -0.254724 0.5225)
+			(end 0.254724 0.5225)
 			(stroke
 				(width 0.12)
@@
 		)
 		(fp_line
-			(start -0.254724 0.5225)
-			(end 0.254724 0.5225)
+			(start -0.254724 -0.5225)
+			(end 0.254724 -0.5225)
 			(stroke
 				(width 0.12)
@@
 		)
 		(fp_line
-			(start -1.65 -0.73)
-			(end 1.65 -0.73)
+			(start -1.65 0.73)
+			(end -1.65 -0.73)
 			(stroke
 				(width 0.05)
@@
 		)
 		(fp_line
-			(start -1.65 0.73)
-			(end -1.65 -0.73)
+			(start 1.65 0.73)
+			(end -1.65 0.73)
 			(stroke
 				(width 0.05)
@@
 		)
 		(fp_line
-			(start 1.65 -0.73)
-			(end 1.65 0.73)
+			(start -1.65 -0.73)
+			(end 1.65 -0.73)
 			(stroke
 				(width 0.05)
@@
 		)
 		(fp_line
-			(start 1.65 0.73)
-			(end -1.65 0.73)
+			(start 1.65 -0.73)
+			(end 1.65 0.73)
 			(stroke
 				(width 0.05)
@@
 		)
 		(fp_line
-			(start -0.8 -0.4125)
-			(end 0.8 -0.4125)
+			(start -0.8 0.4125)
+			(end -0.8 -0.4125)
 			(stroke
 				(width 0.1)
@@
 		)
 		(fp_line
-			(start -0.8 0.4125)
-			(end -0.8 -0.4125)
+			(start 0.8 0.4125)
+			(end -0.8 0.4125)
 			(stroke
 				(width 0.1)
@@
 		)
 		(fp_line
-			(start 0.8 -0.4125)
-			(end 0.8 0.4125)
+			(start -0.8 -0.4125)
+			(end 0.8 -0.4125)
 			(stroke
 				(width 0.1)
@@
 		)
 		(fp_line
-			(start 0.8 0.4125)
-			(end -0.8 0.4125)
+			(start 0.8 -0.4125)
+			(end 0.8 0.4125)
 			(stroke
 				(width 0.1)
@@
 		)
 		(fp_text user "${REFERENCE}"
-			(at 0 0 0)
+			(at 0 0 90)
 			(layer "F.Fab")
 			(effects
@@
 		)
 		(pad "1" smd roundrect
-			(at -0.9125 0)
+			(at -0.9125 0 270)
 			(size 0.975 0.95)
 			(layers "F.Cu" "F.Paste" "F.Mask")
@@
 		)
 		(pad "2" smd roundrect
-			(at 0.9125 0)
+			(at 0.9125 0 270)
 			(size 0.975 0.95)
 			(layers "F.Cu" "F.Paste" "F.Mask")
@@
 	(footprint "Resistor_SMD:R_0603_1608Metric_Pad0.98x0.95mm_HandSolder"
 		(layer "F.Cu")
-		(at 116.2 72 180)
+		(at 113.7 75.0875 -90)
 		(descr "Resistor SMD 0603 (1608 Metric), square (rectangular) end terminal, IPC_7351 nominal with elongated pad for handsoldering. (Body size source: IPC-SM-782 page 72, https://www.pcb-3d.com/wordpress/wp-content/uploads/ipc-sm-782a_amendment_1_and_2.pdf), generated with kicad-footprint-generator")
 		(tags "resistor handsolder")
 		(property "Reference" "R7"
-			(at 0 -1.43 180)
+			(at 0 -1.43 90)
 			(layer "F.SilkS")
 			(effects
@@
 		)
 		(property "Value" "500k"
-			(at 0 1.43 180)
+			(at 0 1.43 90)
 			(layer "F.Fab")
 			(effects
@@
 		)
 		(property "Footprint" "Resistor_SMD:R_0603_1608Metric_Pad0.98x0.95mm_HandSolder"
-			(at 0 0 180)
+			(at 0 0 -90)
 			(unlocked yes)
 			(layer "F.Fab")
@@
 		)
 		(property "Datasheet" ""
-			(at 0 0 180)
+			(at 0 0 -90)
 			(unlocked yes)
 			(layer "F.Fab")
@@
 		)
 		(property "Description" "Resistor, US symbol"
-			(at 0 0 180)
+			(at 0 0 -90)
 			(unlocked yes)
 			(layer "F.Fab")
@@
 		)
 		(fp_line
-			(start 1.65 0.73)
-			(end -1.65 0.73)
+			(start -1.65 0.73)
+			(end -1.65 -0.73)
 			(stroke
 				(width 0.05)
@@
 		)
 		(fp_line
-			(start 1.65 -0.73)
-			(end 1.65 0.73)
+			(start 1.65 0.73)
+			(end -1.65 0.73)
 			(stroke
 				(width 0.05)
@@
 		)
 		(fp_line
-			(start -1.65 0.73)
-			(end -1.65 -0.73)
+			(start -1.65 -0.73)
+			(end 1.65 -0.73)
 			(stroke
 				(width 0.05)
@@
 		)
 		(fp_line
-			(start -1.65 -0.73)
-			(end 1.65 -0.73)
+			(start 1.65 -0.73)
+			(end 1.65 0.73)
 			(stroke
 				(width 0.05)
@@
 		)
 		(fp_line
-			(start 0.8 0.4125)
-			(end -0.8 0.4125)
+			(start -0.8 0.4125)
+			(end -0.8 -0.4125)
 			(stroke
 				(width 0.1)
@@
 		)
 		(fp_line
-			(start 0.8 -0.4125)
-			(end 0.8 0.4125)
+			(start 0.8 0.4125)
+			(end -0.8 0.4125)
 			(stroke
 				(width 0.1)
@@
 		)
 		(fp_line
-			(start -0.8 0.4125)
-			(end -0.8 -0.4125)
+			(start -0.8 -0.4125)
+			(end 0.8 -0.4125)
 			(stroke
 				(width 0.1)
@@
 		)
 		(fp_line
-			(start -0.8 -0.4125)
-			(end 0.8 -0.4125)
+			(start 0.8 -0.4125)
+			(end 0.8 0.4125)
 			(stroke
 				(width 0.1)
@@
 		)
 		(fp_text user "${REFERENCE}"
-			(at 0 0 180)
+			(at 0 0 90)
 			(layer "F.Fab")
 			(effects
@@
 		)
 		(pad "1" smd roundrect
-			(at -0.9125 0 180)
+			(at -0.9125 0 270)
 			(size 0.975 0.95)
 			(layers "F.Cu" "F.Paste" "F.Mask")
@@
 		)
 		(pad "2" smd roundrect
-			(at 0.9125 0 180)
+			(at 0.9125 0 270)
 			(size 0.975 0.95)
 			(layers "F.Cu" "F.Paste" "F.Mask")
@@
 	(footprint "Resistor_SMD:R_0603_1608Metric_Pad0.98x0.95mm_HandSolder"
 		(layer "F.Cu")
-		(at 317.2875 -12.48)
+		(at 113.7 83 -90)
 		(descr "Resistor SMD 0603 (1608 Metric), square (rectangular) end terminal, IPC_7351 nominal with elongated pad for handsoldering. (Body size source: IPC-SM-782 page 72, https://www.pcb-3d.com/wordpress/wp-content/uploads/ipc-sm-782a_amendment_1_and_2.pdf), generated with kicad-footprint-generator")
 		(tags "resistor handsolder")
 		(property "Reference" "R9"
-			(at 0 -1.43 0)
+			(at 0 -1.43 90)
 			(layer "F.SilkS")
 			(effects
@@
 		)
 		(property "Value" "41.7k"
-			(at 0 1.43 0)
+			(at 0 1.43 90)
 			(layer "F.Fab")
 			(effects
@@
 		)
 		(property "Footprint" "Resistor_SMD:R_0603_1608Metric_Pad0.98x0.95mm_HandSolder"
-			(at 0 0 0)
+			(at 0 0 -90)
 			(unlocked yes)
 			(layer "F.Fab")
@@
 		)
 		(property "Datasheet" ""
-			(at 0 0 0)
+			(at 0 0 -90)
 			(unlocked yes)
 			(layer "F.Fab")
@@
 		)
 		(property "Description" "Resistor, US symbol"
-			(at 0 0 0)
+			(at 0 0 -90)
 			(unlocked yes)
 			(layer "F.Fab")
@@
 		)
 		(property "MPN" "RN73R1JTTD4172F10"
-			(at 0 0 0)
+			(at 0 0 -90)
 			(unlocked yes)
 			(layer "F.Fab")
@@
 		)
 		(property "Note" "Vsense"
-			(at 0 0 0)
+			(at 0 0 -90)
 			(unlocked yes)
 			(layer "F.Fab")
@@
 		(attr smd)
 		(fp_line
-			(start -0.254724 -0.5225)
-			(end 0.254724 -0.5225)
+			(start -0.254724 0.5225)
+			(end 0.254724 0.5225)
 			(stroke
 				(width 0.12)
@@
 		)
 		(fp_line
-			(start -0.254724 0.5225)
-			(end 0.254724 0.5225)
+			(start -0.254724 -0.5225)
+			(end 0.254724 -0.5225)
 			(stroke
 				(width 0.12)
@@
 		)
 		(fp_line
-			(start -1.65 -0.73)
-			(end 1.65 -0.73)
+			(start -1.65 0.73)
+			(end -1.65 -0.73)
 			(stroke
 				(width 0.05)
@@
 		)
 		(fp_line
-			(start -1.65 0.73)
-			(end -1.65 -0.73)
+			(start 1.65 0.73)
+			(end -1.65 0.73)
 			(stroke
 				(width 0.05)
@@
 		)
 		(fp_line
-			(start 1.65 -0.73)
-			(end 1.65 0.73)
+			(start -1.65 -0.73)
+			(end 1.65 -0.73)
 			(stroke
 				(width 0.05)
@@
 		)
 		(fp_line
-			(start 1.65 0.73)
-			(end -1.65 0.73)
+			(start 1.65 -0.73)
+			(end 1.65 0.73)
 			(stroke
 				(width 0.05)
@@
 		)
 		(fp_line
-			(start -0.8 -0.4125)
-			(end 0.8 -0.4125)
+			(start -0.8 0.4125)
+			(end -0.8 -0.4125)
 			(stroke
 				(width 0.1)
@@
 		)
 		(fp_line
-			(start -0.8 0.4125)
-			(end -0.8 -0.4125)
+			(start 0.8 0.4125)
+			(end -0.8 0.4125)
 			(stroke
 				(width 0.1)
@@
 		)
 		(fp_line
-			(start 0.8 -0.4125)
-			(end 0.8 0.4125)
+			(start -0.8 -0.4125)
+			(end 0.8 -0.4125)
 			(stroke
 				(width 0.1)
@@
 		)
 		(fp_line
-			(start 0.8 0.4125)
-			(end -0.8 0.4125)
+			(start 0.8 -0.4125)
+			(end 0.8 0.4125)
 			(stroke
 				(width 0.1)
@@
 		)
 		(fp_text user "${REFERENCE}"
-			(at 0 0 0)
+			(at 0 0 90)
 			(layer "F.Fab")
 			(effects
@@
 		)
 		(pad "1" smd roundrect
-			(at -0.9125 0)
+			(at -0.9125 0 270)
 			(size 0.975 0.95)
 			(layers "F.Cu" "F.Paste" "F.Mask")
@@
 		)
 		(pad "2" smd roundrect
-			(at 0.9125 0)
+			(at 0.9125 0 270)
 			(size 0.975 0.95)
 			(layers "F.Cu" "F.Paste" "F.Mask")

Commit message: pushed board
Parts:
- removed TP10: ADC V Sol, TestPoint:TestPoint_THTPad_1.0x1.0mm_Drill0.5mm
- removed TP12: ADC I Sol, TestPoint:TestPoint_THTPad_1.0x1.0mm_Drill0.5mm
- added H1: MountingHole, MountingHole:MountingHole_3.2mm_M3, F.Cu at (71.2, 56.5)
- added H2: MountingHole, MountingHole:MountingHole_3.2mm_M3, F.Cu at (141.2, 56.5)
- added H3: MountingHole, MountingHole:MountingHole_3.2mm_M3, F.Cu at (71.2, 168.0)
- added H4: MountingHole, MountingHole:MountingHole_3.2mm_M3, F.Cu at (141.2, 168.0)
- C27: moved to B.Cu
- JP1: footprint Resistor_SMD:R_0603_1608Metric_Pad0.98x0.95mm_HandSolder -> Resistor_SMD:R_2816_7142Metric
- moved TP13 256.6 mm to (117.2, 129.0)
- moved TP11 234.3 mm to (113.7, 72.0)
- moved TP8 233.1 mm to (138.2, 119.0)
- moved C27 231.6 mm to (129.2, 126.0), turned to 180 degrees
- moved C28 230.1 mm to (129.2, 126.0)
- moved C26 229.2 mm to (134.2, 126.0), turned to 180 degrees
- moved TP6 224.2 mm to (141.7, 119.0)
- moved TP7 214.3 mm to (146.7, 95.5)
- moved TP9 213.6 mm to (143.2, 95.0)
- moved TP2 212.7 mm to (125.2, 61.5)
- moved TP1 212.2 mm to (125.2, 57.0)
- moved TP5 200.7 mm to (143.7, 75.5)
- moved TP3 163.0 mm to (137.2, 95.5)
- moved TP4 158.7 mm to (140.2, 95.5)
- moved C9 28.0 mm to (140.7, 128.5)
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Routing:
- net /Gate: track 0.00 -> 104.5 mm, vias 0 -> 2
- net /Sol In: track 0.00 -> 98.7 mm
- net /ADC I Batt: track 0.00 -> 47.3 mm
- net /ADC V Batt: track 0.00 -> 41.5 mm, vias 0 -> 2
- net /Batt In: track 0.00 -> 39.7 mm
- net /Batt Out: track 0.00 -> 33.8 mm, vias 0 -> 2
- net /Sol Out: track 0.00 -> 32.9 mm
- net +24V: track 3.00 -> 31.0 mm
- net /Board Temp: track 0.00 -> 24.8 mm
- net /ADC V Sol: track 0.00 -> 17.9 mm
- net Net-(U1-+VOUT): track 0.00 -> 16.6 mm, vias 0 -> 1
- net Earth: track 29.4 -> 45.1 mm, vias 2 -> 29
- net Net-(U8-+VIN): track 0.00 -> 15.6 mm
- net GND: track 35.8 -> 50.0 mm, vias 7 -> 13
- net /Sensors/V Sense Batt: track 0.00 -> 14.2 mm
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- added copper zone on F.Cu, net /Batt In
- added copper zone on F.Cu, net /Batt Out
- added copper zone on F.Cu, net /DNP Anode
- added copper zone on F.Cu, net /Sol In
- added copper zone on F.Cu, net /Sol Out
- added copper zone on F.Cu, net Earth
- added copper zone on F.Cu, net Net-(JP1-A)
Other:
- board outline added: 83.6 x 120.1 mm
- board text added: "24V"
- board text added: "3v3"
- board text added: "3v3 HV"
- board text added: "BATTERY INPUT"
- board text added: "GND"
- board text added: "GND HV"
- board text added: "I_Bat"
- board text added: "I_Sol"
- board text added: "Solar Input"
- board text added: "V_Bat"
- board text added: "V_Sol"
