File: HW/PowerBoard_v1/power_v1.kicad_sch (KiCad schematic)
At the start: 27 parts, among them J1 Inputs, J3 Vin Solar, J4 Vout Battery, J5 Sensors, Q201 IXTT220N20X4HV, U120 RO-2412S, U130 STGAP2SMTR

Commit message: updated naming
Connections:
- net Batt Out+ renamed Batt Out
- net CAP + renamed Batt In
- net SHUNT IN renamed Sol Out
- net Solar IN+ renamed Sol In
Other:
- sheet Sensors ports: added Batt In, Batt Out, Sol In, Sol Out; removed Batt Out+, SHUNT IN, SHUNT OUT, Solar IN+
Changed lines of the file:
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@@
 		)
 	)
-	(label "SHUNT IN"
+	(label "Sol Out"
 		(at 128.27 48.26 0)
 		(fields_autoplaced yes)
@@
 		)
 	)
-	(label "ADC V Sol"
-		(at 41.91 171.45 180)
+	(label "Batt Out"
+		(at 116.84 74.93 180)
 		(fields_autoplaced yes)
 		(effects
@@
 		)
 	)
-	(label "DNP Cathode"
-		(at 226.06 113.03 180)
+	(label "Sol In"
+		(at 116.84 62.23 180)
 		(fields_autoplaced yes)
 		(effects
@@
 		)
 	)
-	(label "Solar IN+"
-		(at 116.84 62.23 180)
+	(label "ADC V Sol"
+		(at 41.91 171.45 180)
 		(fields_autoplaced yes)
 		(effects
@@
 		)
 	)
-	(label "Gate"
-		(at 152.4 149.86 180)
+	(label "DNP Cathode"
+		(at 226.06 113.03 180)
 		(fields_autoplaced yes)
 		(effects
@@
 		)
 	)
-	(label "Solar IN+"
-		(at 123.19 48.26 180)
+	(label "Gate"
+		(at 152.4 149.86 180)
 		(fields_autoplaced yes)
 		(effects
@@
 		)
 	)
-	(label "Solar IN-"
-		(at 123.19 50.8 180)
-		(fields_autoplaced yes)
-		(effects
-			(font
-				(size 1.27 1.27)
-			)
-			(justify right bottom)
-		)
-	)
 	(label "ADC I Sol"
 		(at 41.91 166.37 180)
@@
 		)
 	)
-	(label "SHUNT OUT"
-		(at 116.84 72.39 180)
-		(fields_autoplaced yes)
-		(effects
-			(font
-				(size 1.27 1.27)
-			)
-			(justify right bottom)
-		)
-	)
 	(label "Gate"
 		(at 210.82 97.79 0)
@@
 		)
 	)
-	(label "SHUNT OUT"
+	(label "Batt In"
 		(at 223.52 48.26 180)
 		(fields_autoplaced yes)
@@
 		)
 	)
-	(label "Batt Out+"
-		(at 116.84 74.93 180)
+	(label "Sol Out"
+		(at 116.84 64.77 180)
 		(fields_autoplaced yes)
 		(effects
@@
 		)
 	)
-	(label "Batt Out+"
+	(label "Batt Out"
 		(at 228.6 48.26 0)
 		(fields_autoplaced yes)
@@
 		)
 	)
-	(label "SHUNT IN"
-		(at 116.84 64.77 180)
+	(label "Batt In"
+		(at 116.84 72.39 180)
 		(fields_autoplaced yes)
 		(effects
@@
 		)
 	)
-	(label "ADC I Batt"
-		(at 41.91 163.83 180)
+	(label "Sol In"
+		(at 123.19 48.26 180)
 		(fields_autoplaced yes)
 		(effects
@@
 		)
 	)
-	(label "Board Temp"
-		(at 41.91 161.29 180)
+	(label "ADC I Batt"
+		(at 41.91 163.83 180)
 		(fields_autoplaced yes)
 		(effects
@@
 		)
 	)
-	(label "DNP Drain"
-		(at 170.18 52.07 0)
+	(label "Board Temp"
+		(at 41.91 161.29 180)
 		(fields_autoplaced yes)
 		(effects
@@
 				(size 1.27 1.27)
 			)
-			(justify left bottom)
+			(justify right bottom)
 		)
 	)
-	(label "Batt Out-"
-		(at 238.76 50.8 180)
+	(label "DNP Drain"
+		(at 170.18 52.07 0)
 		(fields_autoplaced yes)
 		(effects
@@
 				(size 1.27 1.27)
 			)
-			(justify right bottom)
+			(justify left bottom)
 		)
 	)
@@
 			)
 		)
-		(pin "Batt Out+" output
-			(at 105.41 74.93 0)
+		(pin "Sol In" input
+			(at 105.41 62.23 0)
 			(effects
 				(font
@@
 			)
 		)
-		(pin "SHUNT OUT" input
-			(at 105.41 72.39 0)
+		(pin "Sol Out" output
+			(at 105.41 64.77 0)
 			(effects
 				(font
@@
 			)
 		)
-		(pin "Solar IN+" input
-			(at 105.41 62.23 0)
+		(pin "Batt Out" output
+			(at 105.41 72.39 0)
 			(effects
 				(font
@@
 			)
 		)
-		(pin "SHUNT IN" output
-			(at 105.41 64.77 0)
+		(pin "Batt In" input
+			(at 105.41 74.93 0)
 			(effects
 				(font

Commit message: name changes
Parts:
- removed D3: 0.83V, Package_TO_SOT_SMD:TO-252-2, symbol Device:D_Schottky_AKA
- added D3: 0.83V, Package_TO_SOT_SMD:TO-252-2, symbol device:D_Schottky_AKA
- D2: symbol Device:D_Schottky_AKA -> device:D_Schottky_AKA
Connections:
- net Batt In: now also D3.2 (K)
- net DNP Anode: now also D3.1 (A), D3.3 (A)

Commit message: more changes
Connections:
- net +3V3: now also J1.2 (Pin_2); no longer J1.4 (Pin_4)
- net ADC I Batt: now also J5.1 (Pin_1); no longer J5.4 (Pin_4)
- net ADC I Sol: now also J5.5 (Pin_5); no longer J5.3 (Pin_3)
- net ADC V Sol: now also J5.4 (Pin_4); no longer J5.1 (Pin_1)
- net Board Temp: now also J5.3 (Pin_3); no longer J5.5 (Pin_5)
- net PWM: now also J1.4 (Pin_4); no longer J1.2 (Pin_2)

Commit message: pushed board
Parts:
- added H1, H2, H3, H4: MountingHole, MountingHole:MountingHole_3.2mm_M3, symbol Mechanical:MountingHole
- JP1: footprint Resistor_SMD:R_0603_1608Metric_Pad0.98x0.95mm_HandSolder -> Resistor_SMD:R_2816_7142Metric
