File: HW/LogicBoard_v1/LogicBoard_v1_CAN.kicad_sch (KiCad schematic)
At the start: 0 parts

Commit message: Finsihed logic board schematic
Parts:
- added C10, C11, C12, C14: 0.1μF, Capacitor_SMD:C_0603_1608Metric_Pad1.08x0.95mm_HandSolder, symbol device:C
- added C13, C8: 10μF, Capacitor_SMD:C_1206_3216Metric_Pad1.33x1.80mm_HandSolder, symbol device:C
- added C9: 1μF, Capacitor_SMD:C_0805_2012Metric_Pad1.18x1.45mm_HandSolder, symbol device:C
- added D7: PESD1CAN, Package_TO_SOT_SMD:SOT-23, symbol Discrete_SMD:PESD1CAN
- added D8: Yellow, LED_SMD:LED_0603_1608Metric_Pad1.05x0.95mm_HandSolder, symbol device:LED
- added F2: 0.2A, Fuse:Fuse_1206_3216Metric_Pad1.42x1.75mm_HandSolder, symbol Discrete_SMD:Polyfuse
- added J5: CAN, layout:M12_5-pin_90deg_VertPitch2.54mm, symbol Connector_Generic:Conn_01x05
- added R11: 1M, Resistor_SMD:R_0603_1608Metric_Pad0.98x0.95mm_HandSolder, symbol device:R
- added R12: 120, Resistor_SMD:R_1206_3216Metric_Pad1.30x1.75mm_HandSolder, symbol device:R
- added R13: 1k, Resistor_SMD:R_0603_1608Metric_Pad0.98x0.95mm_HandSolder, symbol device:R
- added S1: CL-SB-22B-01, layout:DPDT_NIDEC_6_pin_SMD_1.6_x_1.2_pads, symbol Misc:CL-SB-22A
- added TP5: CAN_VCC_Fused, TestPoint:TestPoint_Pad_1.0x1.0mm, symbol Connector:TestPoint
- added TP6: GND_CAN, TestPoint:TestPoint_Pad_1.0x1.0mm, symbol Connector:TestPoint
- added TP7: +5V_CAN, TestPoint:TestPoint_Pad_1.0x1.0mm, symbol Connector:TestPoint
- added U3: MCP1754S-5002E_SOT23A, Package_TO_SOT_SMD:SOT-23, symbol Regulator_Linear:MCP1700-5002E_SOT23
- added U4: ISO1042DWV, layout:SOIC-8_5.85x7.4mm_P1.27mm, symbol ICs:ISO1042DWV
Connections:
- net CAN_RX: now also U4.3 (RXD)
- net CAN_TX: now also U4.2 (TXD)
- new net: D8.2 (A), R13.1
- new net: R12.1, S1.6
- new net +3V3: C10.1, C8.1, C9.1, U4.1 (Vcc1)
- new net +5V_CAN: C12.1, C13.1, C14.1, R13.2, TP7.1, U3.2 (VO), U4.8 (Vcc2)
- new net CANH: D7.2 (K), J5.4 (Pin_4), S1.5, U4.7 (CANH)
- new net CANL: D7.1 (K), J5.5 (Pin_5), R12.2, U4.6 (CANL)
- new net CAN_Shield: J5.1 (Pin_1), R11.2
- new net CAN_VCC_Fused: C11.1, F2.1, TP5.1, U3.3 (VI)
- new net CAN_VCC_Unfused: F2.2, J5.2 (Pin_2)
- new net GND: C10.2, C8.2, C9.2, U4.4 (GND1)
- new net GND_CAN: C11.2, C12.2, C13.2, C14.2, D7.3 (A), J5.3 (Pin_3), R11.1, S1.3, TP6.1, U3.1 (GND), U4.5 (GND2)
- new net TERM_LED: D8.1 (K), S1.2
- no-connect marks 0 -> 2
Other:
- note added: "12V regulator"
- note added: "ESD protect"
- note added: "Isolation to/from rest of board"
- note added: "Optional termination"

Commit message: Started logic board
Parts:
- C10: renamed from C11; value 0.1μF -> 0.1uF
- C11: renamed from C12; value 0.1μF -> 0.1uF
- C12: renamed from C13; value 10μF -> 10uF
- C13: renamed from C14; value 0.1μF -> 0.1uF
- C7: renamed from C8; value 10μF -> 10uF
- C8: renamed from C9; value 1μF -> 1uF
- C9: renamed from C10; value 0.1μF -> 0.1uF
- TP2: renamed from TP5; footprint TestPoint:TestPoint_Pad_1.0x1.0mm -> TestPoint:TestPoint_THTPad_D1.5mm_Drill0.7mm
- TP3: renamed from TP6; footprint TestPoint:TestPoint_Pad_1.0x1.0mm -> TestPoint:TestPoint_THTPad_D1.5mm_Drill0.7mm
- TP4: renamed from TP7; footprint TestPoint:TestPoint_Pad_1.0x1.0mm -> TestPoint:TestPoint_THTPad_D1.5mm_Drill0.7mm
- renumbered D7 to D1, D8 to D2, F2 to F1, J5 to J6, R11 to R7, R12 to R8, R13 to R9, U3 to U2, U4 to U3
Other:
- company: (none) -> Illini Solar Car
- title: (none) -> MPPT Logic Board
