File: HW/LogicBoard_v1/LogicBoard_v1_Fans.kicad_sch (KiCad schematic)
At the start: 22 parts, among them J6 Fans, Q3 Q_NMOS_GSD, U5 BD450M2FP3-CE2

Commit message: Started logic board
Parts:
- removed TP11: TestPoint, TestPoint:TestPoint_Pad_1.0x1.0mm, symbol Connector:TestPoint
- removed TP9: Test Point, TestPoint:TestPoint_Pad_1.0x1.0mm, symbol Connector:TestPoint
- C17: renamed from C15; value 0.1µ -> 0.1uF; Note 10V X5R 0603 -> (none)
- J7: renamed from J6; MPN SCT2541 -> (none)
- R13: renamed from R14; Note 0.1W 5% 0603 -> (none)
- TP10: renamed from TP12; value TestPoint -> Fan PWM; footprint TestPoint:TestPoint_Pad_1.0x1.0mm -> TestPoint:TestPoint_THTPad_D1.5mm_Drill0.7mm
- TP9: renamed from TP8; footprint TestPoint:TestPoint_THTPad_D1.0mm_Drill0.5mm -> TestPoint:TestPoint_THTPad_D1.5mm_Drill0.7mm
- renumbered C16 to C15, C17 to C16, D11 to D10, D10 to D8, R15 to R14, R17 to R15
Other:
- company: (none) -> Illini Solar Car
- title: (none) -> MPPT Logic Board
