File: HW/LogicBoard_v1/LogicBoard_v1_MCU.kicad_sch (KiCad schematic)
At the start: 17 parts, among them J1 JTAG_Header, U1 LPC1547JBD48, Y1 12MHz

Commit message: Finsihed logic board schematic
Parts:
- gave numbers to parts that had none: 14
Connections:
- net Fan_Tach: now reaches U1.6 (PIO0_5/ADC0_3)
- net Fan_PWM: now reaches U1.7 (PIO0_6/ADC0_2/SCT2_OUT3)

Commit message: Started logic board
Parts:
- added C19, C20: 0.1uF, Capacitor_SMD:C_0603_1608Metric_Pad1.08x0.95mm_HandSolder, symbol device:C
- C1: renamed from C2; footprint Capacitor_SMD:C_0603_1608Metric -> Capacitor_SMD:C_0603_1608Metric_Pad1.08x0.95mm_HandSolder; Note 10V X5R 0603 20% -> (none)
- C2: renamed from C3; footprint Capacitor_SMD:C_0603_1608Metric -> Capacitor_SMD:C_0603_1608Metric_Pad1.08x0.95mm_HandSolder; Note 10V X5R 0603 20% -> (none)
- C3: renamed from C4; footprint Capacitor_SMD:C_0603_1608Metric -> Capacitor_SMD:C_0603_1608Metric_Pad1.08x0.95mm_HandSolder; Note 10V X5R 0603 20% -> (none)
- C4: renamed from C5; footprint Capacitor_SMD:C_0603_1608Metric -> Capacitor_SMD:C_0603_1608Metric_Pad1.08x0.95mm_HandSolder; Note 10V X5R 0603 20% -> (none)
- C5: renamed from C6; footprint Capacitor_SMD:C_0603_1608Metric -> Capacitor_SMD:C_0603_1608Metric_Pad1.08x0.95mm_HandSolder; Note 10V X5R 0603 20% -> (none)
- C6: renamed from C7; footprint Capacitor_SMD:C_0603_1608Metric -> Capacitor_SMD:C_0603_1608Metric_Pad1.08x0.95mm_HandSolder; Note 10V X5R 0603 20% -> (none)
- R1: renamed from R5; footprint Resistor_SMD:R_0603_1608Metric -> Resistor_SMD:R_0603_1608Metric_Pad0.98x0.95mm_HandSolder; Note 0.1W 5% 0603 -> (none)
- R2: renamed from R6; footprint Resistor_SMD:R_0603_1608Metric -> Resistor_SMD:R_0603_1608Metric_Pad0.98x0.95mm_HandSolder; Note 0.1W 5% 0603 -> (none)
- R3: renamed from R7; footprint Resistor_SMD:R_0603_1608Metric -> Resistor_SMD:R_0603_1608Metric_Pad0.98x0.95mm_HandSolder; Note 0.1W 5% 0603 -> (none)
- R4: renamed from R8; footprint Resistor_SMD:R_0603_1608Metric -> Resistor_SMD:R_0603_1608Metric_Pad0.98x0.95mm_HandSolder; Note 0.1W 5% 0603 -> (none)
- R5: renamed from R9; footprint Resistor_SMD:R_0603_1608Metric -> Resistor_SMD:R_0603_1608Metric_Pad0.98x0.95mm_HandSolder; Note 0.1W 5% 0603 -> (none)
- R6: renamed from R10; footprint Resistor_SMD:R_0603_1608Metric -> Resistor_SMD:R_0603_1608Metric_Pad0.98x0.95mm_HandSolder; Note 0.1W 5% 0603 -> (none)
- SW1, SW2: footprint layout:RST_STM_PTS_820_Series -> layout:Button_223AM; MPN ADTSM31NV -> 223AMVAAR
- U1: footprint Housings_QFP:LQFP-48_7x7mm_Pitch0.5mm -> Package_QFP:LQFP-48_7x7mm_P0.5mm
- renumbered J1 to J5
Connections:
- net GND: now also Y1.2, Y1.4, C19.2, C20.2
- net VCC: now also C19.1
- net ADC_3: now reaches U1.22 (PIO0_14/ADC1_7/SCT1_OUT5)
- net ADC_4: now reaches U1.23 (PIO0_15/ADC1_8)
- net ADC_1: now reaches U1.4 (PIO0_3/ADC0_5/SCT1_OUT4)
- net ADC_2: now reaches U1.8 (PIO0_7/ADC0_1)
- net P0_16 renamed ISP1
- net P0_21 renamed RESET
- net RESET: now also C20.1
- net P0_4 renamed ISP0
- net Temp_Sens renamed Temp_Sens_ADC
- no-connect marks 5 -> 12
Other:
- note removed: "0.1uF near VDDA"
- note removed: "Pair of 0.1uF near VDD"
- company: (none) -> Illini Solar Car
- title: (none) -> MPPT Logic Board
