File: HW/LogicBoard_v1/LogicBoard_v1_Power.kicad_sch (KiCad schematic)
At the start: 17 parts, among them Q1 Q_PMOS_GDS, Q2 Q_PMOS_GDS

Commit message: Finsihed logic board schematic
Parts:
- removed TP4: VGS Threshold, TestPoint:TestPoint_THTPad_D1.5mm_Drill0.7mm, symbol Connector:TestPoint
- added D6: D_Schottky, Diode_SMD:D_SOD-123F, symbol device:D_Schottky
- added U2: R-783.3-0.5, Converter_DCDC:Converter_DCDC_RECOM_R-78E-0.5_THT, symbol Regulator_Switching:R-783.3-0.5
Connections:
- net +24V_FUSED: now also TP1.1
- net 24V_Protected: now also TP2.1, D6.1 (K), U2.1 (IN)
- net 3v3: now also D6.2 (A), U2.3 (OUT)
- net GND: now also U2.2 (GND)
- net at Q1.1 (G), Q2.1 (G), R1.1: now also D2.2 (A)
Other:
- moved on the sheet: D2, D4, TP1, TP2

Commit message: Started logic board
Parts:
- removed D4: LED, LED_SMD:LED_0603_1608Metric_Pad1.05x0.95mm_HandSolder, symbol device:LED
- removed R3: 10k, Resistor_SMD:R_0603_1608Metric_Pad1.05x0.95mm_HandSolder, symbol device:R
- added TP8: 3v3, TestPoint:TestPoint_THTPad_D1.5mm_Drill0.7mm, symbol Connector:TestPoint
- C14: renamed from C1; footprint Capacitor_SMD:C_0603_1608Metric_Pad1.05x0.95mm_HandSolder -> Capacitor_SMD:C_0603_1608Metric_Pad1.08x0.95mm_HandSolder
- F2: renamed from F1; Notes 32V 125°C 0603 -> (none)
- Q1, Q2: Notes 30Vgs 9.4A 2.5W 150°C max -> (none)
- R10: renamed from R1; footprint Resistor_SMD:R_0603_1608Metric_Pad1.05x0.95mm_HandSolder -> Resistor_SMD:R_0603_1608Metric_Pad0.98x0.95mm_HandSolder; Notes 0.1W 1% 0603 -> (none)
- R11: renamed from R2; footprint Resistor_SMD:R_0603_1608Metric_Pad1.05x0.95mm_HandSolder -> Resistor_SMD:R_0603_1608Metric_Pad0.98x0.95mm_HandSolder; Notes 0.1W 1% 0603 -> (none)
- R12: renamed from R4; footprint Resistor_SMD:R_0603_1608Metric_Pad1.05x0.95mm_HandSolder -> Resistor_SMD:R_0603_1608Metric_Pad0.98x0.95mm_HandSolder; Notes 0.1W 1% 0603 -> (none)
- U4: renamed from U2; MPN (none) -> R-783.3-0.5
- renumbered D1 to D3, D2 to D4, D3 to D5, D5 to D6, D6 to D7, TP1 to TP5, TP3 to TP6, TP2 to TP7
Connections:
- net 3v3: now also TP8.1
- net GND: now also TP6.1
Other:
- company: (none) -> Illini Solar Car
- title: (none) -> MPPT Logic Board
- moved on the sheet: TP6
