File: HW/LogicBoard_v1/LogicBoard_v1.kicad_pcb (KiCad board)
At the start: 2 copper layers, 0 parts

Commit message: Started logic board
Parts:
- added C1: 0.1uF, Capacitor_SMD:C_0603_1608Metric_Pad1.08x0.95mm_HandSolder, F.Cu at (122.7, 109.6)
- added C10: 0.1uF, Capacitor_SMD:C_0603_1608Metric_Pad1.08x0.95mm_HandSolder, F.Cu at (-70.2, -49.4)
- added C11: 0.1uF, Capacitor_SMD:C_0603_1608Metric_Pad1.08x0.95mm_HandSolder, F.Cu at (-70.2, -46.9)
- added C12: 10uF, Capacitor_SMD:C_1206_3216Metric_Pad1.33x1.80mm_HandSolder, F.Cu at (-61.5, -48.1)
- added C13: 0.1uF, Capacitor_SMD:C_0603_1608Metric_Pad1.08x0.95mm_HandSolder, F.Cu at (-70.2, -44.4)
- added C14: 0.047u, Capacitor_SMD:C_0603_1608Metric_Pad1.08x0.95mm_HandSolder, F.Cu at (148.2, 67.2)
- added C15: 0.1uF, Capacitor_SMD:C_0603_1608Metric_Pad1.08x0.95mm_HandSolder, F.Cu at (-93.1, 21.2)
- added C16: 10uF, Capacitor_SMD:C_0603_1608Metric_Pad1.08x0.95mm_HandSolder, F.Cu at (-93.1, 23.7)
- added C17: 0.1uF, Capacitor_SMD:C_0603_1608Metric_Pad1.08x0.95mm_HandSolder, F.Cu at (-93.1, 26.2)
- added C18: 1uF, Capacitor_SMD:C_0603_1608Metric_Pad1.08x0.95mm_HandSolder, F.Cu at (-93.1, 28.7)
- added C19: 0.1uF, Capacitor_SMD:C_0603_1608Metric_Pad1.08x0.95mm_HandSolder, B.Cu at (132.7, 107.0)
- added C2: 0.1uF, Capacitor_SMD:C_0603_1608Metric_Pad1.08x0.95mm_HandSolder, F.Cu at (127.3, 112.8)
- added C20: 0.1uF, Capacitor_SMD:C_0603_1608Metric_Pad1.08x0.95mm_HandSolder, B.Cu at (132.7, 103.6)
- added C3: 0.1uF, Capacitor_SMD:C_0603_1608Metric_Pad1.08x0.95mm_HandSolder, F.Cu at (131.3, 100.8)
- added C4: 0.1uF, Capacitor_SMD:C_0603_1608Metric_Pad1.08x0.95mm_HandSolder, F.Cu at (127.9, 100.8)
- added C5: 18pF, Capacitor_SMD:C_0603_1608Metric_Pad1.08x0.95mm_HandSolder, F.Cu at (139.5, 107.4)
- added C6: 18pF, Capacitor_SMD:C_0603_1608Metric_Pad1.08x0.95mm_HandSolder, F.Cu at (139.3, 111.4)
- added C7: 10uF, Capacitor_SMD:C_1206_3216Metric_Pad1.33x1.80mm_HandSolder, F.Cu at (-61.5, -51.5)
- added C8: 1uF, Capacitor_SMD:C_0805_2012Metric_Pad1.18x1.45mm_HandSolder, F.Cu at (-92.1, -21.0)
- added C9: 0.1uF, Capacitor_SMD:C_0603_1608Metric_Pad1.08x0.95mm_HandSolder, F.Cu at (-70.2, -51.9)
- added D1: PESD1CAN, Package_TO_SOT_SMD:SOT-23, F.Cu at (-62.2, -35.9)
- added D10: 40V 2A, Diode_SMD:D_1206_3216Metric_Pad1.42x1.75mm_HandSolder, F.Cu at (-81.9, 42.6)
- added D2: Yellow, LED_SMD:LED_0603_1608Metric_Pad1.05x0.95mm_HandSolder, F.Cu at (-87.5, -21.2)
- added D3: Q_SCR_KAG, Package_TO_SOT_SMD:SOT-223-3_TabPin2, F.Cu at (150.4, 73.4)
- added D4: 20 V, Diode_SMD:D_SOD-123F, F.Cu at (160.2, 90.8)
- added D5: 28 V, Diode_SMD:D_SOD-123F, F.Cu at (145.6, 76.8)
- added D6: LED, LED_SMD:LED_0603_1608Metric_Pad1.05x0.95mm_HandSolder, F.Cu at (150.8, 83.8)
- added D7: D_Schottky, Diode_SMD:D_SOD-123F, F.Cu at (148.6, 99.8)
- added D8: 3V6, Diode_SMD:D_SOD-123F, F.Cu at (-88.2, 39.3)
- added D9: 3V6, Diode_SMD:D_SOD-123F, F.Cu at (-88.2, 42.6)
- added F1: 0.2A, Fuse:Fuse_1206_3216Metric_Pad1.42x1.75mm_HandSolder, F.Cu at (-61.5, -44.8)
- added F2: 5A, layout:Littelfuse_154_4.24mm_x_3.81mm, F.Cu at (158.0, 69.2)
- added F3: 100mA, Fuse:Fuse_2512_6332Metric, F.Cu at (-80.6, 38.4)
- added F4: 0.25A Fuse, Fuse:Fuse_1206_3216Metric_Pad1.42x1.75mm_HandSolder, F.Cu at (-87.9, 29.4)
- added F5: 0.2A Fuse, Fuse:Fuse_1206_3216Metric_Pad1.42x1.75mm_HandSolder, F.Cu at (-87.9, 32.7)
- added F6: 1A Fuse, Fuse:Fuse_1206_3216Metric_Pad1.42x1.75mm_HandSolder, F.Cu at (-87.9, 36.0)
- added J1: 24V In, Connector_Molex:Molex_Micro-Fit_3.0_43650-0300_1x03_P3.00mm_Horizontal, F.Cu at (164.0, 63.0)
- added J2: Comm, Connector_Molex:Molex_Micro-Fit_3.0_43650-0600_1x06_P3.00mm_Horizontal, F.Cu at (27.4, 63.3)
- added J3: ADC, Connector_Molex:Molex_Micro-Fit_3.0_43650-0500_1x05_P3.00mm_Horizontal, F.Cu at (27.4, 75.3)
- added J4: Power, Connector_Molex:Molex_Micro-Fit_3.0_43650-0400_1x04_P3.00mm_Horizontal, F.Cu at (164.0, 97.7)
- added J5: JTAG_Header, layout:IDC-Header_2x05_Pitch1.27mm_Straight, F.Cu at (138.8, 98.4)
- added J6: CAN, layout:M12_5-pin_90deg_VertPitch2.54mm, F.Cu at (-83.4, -45.8)
- added J7: Fans, Connector_Molex:Molex_KK-254_AE-6410-04A_1x04_P2.54mm_Vertical, F.Cu at (-86.2, 15.7)
- added Q1: Q_PMOS_GDS, Package_TO_SOT_SMD:TO-252-2, F.Cu at (157.6, 80.8)
- added Q2: Q_PMOS_GDS, Package_TO_SOT_SMD:TO-252-2, F.Cu at (153.4, 90.0)
- added Q3: Q_NMOS_GSD, Package_TO_SOT_SMD:SOT-23_Handsoldering, F.Cu at (-75.5, 22.2)
- added R1: 10k, Resistor_SMD:R_0603_1608Metric_Pad0.98x0.95mm_HandSolder, F.Cu at (121.1, 107.6)
- added R10: 1k, Resistor_SMD:R_0603_1608Metric_Pad0.98x0.95mm_HandSolder, F.Cu at (160.2, 94.8)
- added R11: 10k, Resistor_SMD:R_0603_1608Metric_Pad0.98x0.95mm_HandSolder, F.Cu at (146.6, 67.2)
- added R12: 10k, Resistor_SMD:R_0603_1608Metric_Pad0.98x0.95mm_HandSolder, F.Cu at (150.8, 85.6)
- added R13: 10k, Resistor_SMD:R_0603_1608Metric_Pad0.98x0.95mm_HandSolder, F.Cu at (-93.1, 31.2)
- added R14: 500, Resistor_SMD:R_0603_1608Metric_Pad0.98x0.95mm_HandSolder, F.Cu at (-93.1, 33.7)
- added R15: 10k, Resistor_SMD:R_0603_1608Metric_Pad0.98x0.95mm_HandSolder, F.Cu at (-93.1, 36.2)
- added R16: 10K, Resistor_SMD:R_0603_1608Metric_Pad0.98x0.95mm_HandSolder, F.Cu at (-93.1, 38.7)
- added R2: 10k, Resistor_SMD:R_0603_1608Metric_Pad0.98x0.95mm_HandSolder, F.Cu at (129.5, 119.6)
- added R3: 1k, Resistor_SMD:R_0603_1608Metric_Pad0.98x0.95mm_HandSolder, F.Cu at (135.3, 117.6)
- added R4: 0, Resistor_SMD:R_0603_1608Metric_Pad0.98x0.95mm_HandSolder, F.Cu at (142.9, 102.0)
- added R5: 10k, Resistor_SMD:R_0603_1608Metric_Pad0.98x0.95mm_HandSolder, F.Cu at (126.7, 95.6)
- added R6: 1k, Resistor_SMD:R_0603_1608Metric_Pad0.98x0.95mm_HandSolder, F.Cu at (134.9, 91.0)
- added R7: 1M, Resistor_SMD:R_0603_1608Metric_Pad0.98x0.95mm_HandSolder, F.Cu at (-70.2, -41.9)
- added R8: 120, Resistor_SMD:R_1206_3216Metric_Pad1.30x1.75mm_HandSolder, F.Cu at (-61.5, -41.5)
- added R9: 1k, Resistor_SMD:R_0603_1608Metric_Pad0.98x0.95mm_HandSolder, F.Cu at (-70.2, -39.4)
- added S1: CL-SB-22B-01, layout:DPDT_NIDEC_6_pin_SMD_1.6_x_1.2_pads, F.Cu at (-68.5, -32.9)
- added SW1: ISP, layout:Button_223AM, F.Cu at (132.3, 115.8)
- added SW2: ~RESET, layout:Button_223AM, F.Cu at (132.1, 94.8)
- added TP1: Duty PWM, TestPoint:TestPoint_THTPad_D1.5mm_Drill0.7mm, F.Cu at (160.6, 105.6)
- added TP10: Fan PWM, TestPoint:TestPoint_THTPad_D1.5mm_Drill0.7mm, F.Cu at (-74.5, 41.3)
- added TP2: CAN_VCC_Fused, TestPoint:TestPoint_THTPad_D1.5mm_Drill0.7mm, F.Cu at (-66.2, -51.4)
- added TP3: GND_CAN, TestPoint:TestPoint_THTPad_D1.5mm_Drill0.7mm, F.Cu at (-66.2, -47.8)
- added TP4: +5V_CAN, TestPoint:TestPoint_THTPad_D1.5mm_Drill0.7mm, F.Cu at (-66.2, -44.3)
- added TP5: 24V IN, TestPoint:TestPoint_THTPad_D1.5mm_Drill0.7mm, F.Cu at (162.6, 74.4)
- added TP6: GND, TestPoint:TestPoint_THTPad_D1.5mm_Drill0.7mm, F.Cu at (145.0, 95.0)
- added TP7: 24V OUT, TestPoint:TestPoint_THTPad_D1.5mm_Drill0.7mm, F.Cu at (145.0, 88.6)
- added TP8: 3v3, TestPoint:TestPoint_THTPad_D1.5mm_Drill0.7mm, F.Cu at (145.0, 100.6)
- added TP9: Tach, TestPoint:TestPoint_THTPad_D1.5mm_Drill0.7mm, F.Cu at (-74.5, 37.8)
- added U1: LPC1547JBD48, Package_QFP:LQFP-48_7x7mm_P0.5mm, F.Cu at (128.6, 106.8)
- added U2: MCP1754S-5002E_SOT23A, Package_TO_SOT_SMD:SOT-23, F.Cu at (-62.2, -31.4)
- added U3: ISO1042DWV, layout:SOIC-8_5.85x7.4mm_P1.27mm, F.Cu at (-65.4, -24.1)
- added U4: R-783.3-0.5, Converter_DCDC:Converter_DCDC_RECOM_R-78E-0.5_THT, F.Cu at (152.2, 97.2)
- added U5: BD450M2FP3-CE2, Package_TO_SOT_SMD:SOT-223-3_TabPin2, F.Cu at (-80.0, 31.9)
- added Y1: 12MHz, layout:Crystal_SMD_TXC_7M-4pin_3.2x2.5mm, F.Cu at (137.5, 109.6)
Routing:
- net +24V: track 0.00 -> 42.9 mm
- net /MCU/PWM: track 0.00 -> 42.2 mm, vias 0 -> 2
- net /MCU/RESET: track 0.00 -> 25.4 mm, vias 0 -> 1
- net +3V3: track 0.00 -> 21.0 mm, vias 0 -> 1
- net /Power/+24V_FUSED: track 0.00 -> 20.9 mm
- net Net-(J5-TDO): track 0.00 -> 18.6 mm, vias 0 -> 3
- net GND: track 0.00 -> 15.9 mm, vias 0 -> 6
- net Net-(D4-A): track 0.00 -> 12.5 mm
- net /MCU/TCLK: track 0.00 -> 10.9 mm, vias 0 -> 2
- net Net-(D3-G): track 0.00 -> 10.7 mm
- net /MCU/ISP1: track 0.00 -> 9.61 mm
- net Net-(U1-XTALIN): track 0.00 -> 7.84 mm
- net /MCU/TMS: track 0.00 -> 7.83 mm
- net Net-(R3-Pad2): track 0.00 -> 7.79 mm
- net Net-(R6-Pad2): track 0.00 -> 7.64 mm
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- added copper zone on F.Cu, net +3V3
- added copper zone on B.Cu, net GND
- added copper zone on F.Cu, net GND
- added copper zone on F.Cu, net Net-(D4-K)
Other:
- board outline added: 85 x 100.2 mm
- board text added: "+"
- board text added: "+24V"
- board text added: "+3v3"
- board text added: "-"
- board text added: "24V BUS"
- board text added: "24V_In"
- board text added: "GND"
- board text added: "PGRM"
- board text added: "PWM"

Commit message: Almost done with logic board
Parts:
- C18, C7, C8, C9: moved to B.Cu
- moved C9 257.1 mm to (125.4, 115.0), turned to 90 degrees
- moved C8 254.2 mm to (122.6, 115.0), turned to 90 degrees
- moved C7 245.8 mm to (119.4, 115.0), turned to 90 degrees
- moved C10 242.5 mm to (103.0, 120.4)
- moved C11 242.0 mm to (105.8, 119.2), turned to -90 degrees
- moved J6 241.0 mm to (94.1, 117.2), turned to -90 degrees
- moved C15 240.9 mm to (138.6, 87.0), turned to 180 degrees
- moved C16 239.8 mm to (140.4, 78.2), turned to 180 degrees
- moved R16 236.5 mm to (140.4, 76.6), turned to 180 degrees
- moved C13 235.7 mm to (104.2, 114.2), turned to 90 degrees
- moved R7 235.2 mm to (98.2, 122.4), turned to 180 degrees
- moved F4 234.1 mm to (141.8, 74.4), turned to 180 degrees
- moved C12 233.9 mm to (106.2, 115.0), turned to 90 degrees
- moved C18 230.4 mm to (134.6, 64.0)
- moved C17 229.6 mm to (130.4, 78.6), turned to 90 degrees
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Routing:
- net /Fans/Fan_Tach: track 0.00 -> 44.3 mm, vias 0 -> 2
- net GND: track 15.9 -> 48.6 mm, vias 6 -> 16
- net /Fans/Fan_PWM: track 0.00 -> 26.2 mm, vias 0 -> 4
- net /Fans/PWM_5V: track 0.00 -> 21.7 mm
- net /Fans/24V_fused: track 0.00 -> 21.7 mm
- net +24V: track 42.9 -> 64.0 mm
- net Net-(J7-Pin_1): track 0.00 -> 17.4 mm
- net /Fans/Tach: track 0.00 -> 14.8 mm
- net /Power/+24V_FUSED: track 20.9 -> 26.3 mm
- net +5V: track 0.00 -> 4.01 mm
- net Net-(J7-Pin_4): track 0.00 -> 3.22 mm
- net Net-(F3-Pad1): track 0.00 -> 2.81 mm
- net Net-(Q3-G): track 0.00 -> 2.16 mm
- net /MCU/PWM: vias 2 -> 1
Other:
- board size 85 x 100.2 mm -> 85 x 70 mm
- board text added: "24V"
- board text added: "3V3"
- board text added: "FAN"
- board text added: "Power Out"
- board text added: "Tach"

Commit message: Finsihed logic board
Parts:
- added H1: MountingHole, MountingHole:MountingHole_3.2mm_M3, F.Cu at (92.0, 62.0)
- added H2: MountingHole, MountingHole:MountingHole_3.2mm_M3, F.Cu at (169.0, 124.0)
- C12: moved to B.Cu
- moved J2 73.2 mm to (100.5, 67.0)
- moved J3 71.5 mm to (97.0, 91.6), turned to 90 degrees
- moved TP2 42.6 mm to (103.2, 126.0)
- moved TP4 42.0 mm to (107.0, 126.0)
- moved TP3 37.1 mm to (99.0, 126.0)
- moved C15 6.35 mm to (144.2, 84.0), turned to 90 degrees
- moved R5 4.06 mm to (130.2, 97.6), turned to 0 degrees
- moved D9 3.86 mm to (126.8, 89.0), turned to 90 degrees
- moved F3 2.60 mm to (123.6, 87.4)
- moved C12 2.40 mm to (108.6, 115.0)
Routing:
- net /MCU/Temp_Sens_ADC: track 0.00 -> 73.2 mm
- net /MCU/ADC_4: track 0.00 -> 56.5 mm, vias 0 -> 5
- net /MCU/MISO: track 0.00 -> 55.7 mm, vias 0 -> 4
- net /MCU/SCLK: track 0.00 -> 54.7 mm, vias 0 -> 4
- net /MCU/MOSI: track 0.00 -> 54.2 mm, vias 0 -> 4
- net /MCU/ADC_3: track 0.00 -> 49.1 mm, vias 0 -> 3
- net /MCU/CS_2: track 0.00 -> 44.0 mm, vias 0 -> 2
- net /MCU/CS_1: track 0.00 -> 43.0 mm, vias 0 -> 2
- net /MCU/ADC_2: track 0.00 -> 41.8 mm, vias 0 -> 2
- net /CAN/CANH: track 0.00 -> 40.0 mm, vias 0 -> 3
- net /CAN/+5V_CAN: track 0.00 -> 39.9 mm, vias 0 -> 1
- net /MCU/ADC_1: track 0.00 -> 35.8 mm, vias 0 -> 2
- net /CAN/CANL: track 0.00 -> 25.3 mm, vias 0 -> 2
- net /CAN/CAN_VCC_Fused: track 0.00 -> 15.5 mm
- net /CAN/GND_CAN: track 0.00 -> 15.0 mm, vias 0 -> 5
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- added copper zone on B.Cu, net /CAN/GND_CAN
Other:
- outline, holes or cut-outs redrawn
- board text added: "<- TERM"
- board text added: "ADC"
- board text added: "ADC1"
- board text added: "ADC2"
- board text added: "ADC3"
- board text added: "ADC4"
- board text added: "CS1"
- board text added: "CS2"
- board text added: "Logic Board v1.0"
- board text added: "MISO"
- board text added: "MOSI"
- board text added: "RST"
- board text added: "SCLK"
- board text added: "SPI"
- board text added: "Team #25 Alex Chmiel Alex Lymberopoulos Akhil Pothineni"
- board text added: "Temp"
