File: HW/LogicBoard_v1/LogicBoard_v1.kicad_sch (KiCad schematic)
At the start: 3 parts, among them J2 24V In, J3 Comm, J4 Power

Commit message: Finsihed logic board schematic
Other:
- added sheet Fans (LogicBoard_v1_Fans.kicad_sch)
- sheet MCU ports: added Fan_PWM, Fan_Tach; removed none
- moved on the sheet: J2
Changed lines of the file:
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@@
   (junction (at 105.41 66.548) (diameter 0) (color 0 0 0 0)
   )
-  (junction (at 28.956 49.022) (diameter 0) (color 0 0 0 0)
+  (junction (at 42.926 49.022) (diameter 0) (color 0 0 0 0)
   )
   (wire (pts (xy 101.092 49.276) (xy 101.092 36.322))
@@
     (stroke (width 0) (type default))
   )
-  (wire (pts (xy 26.924 43.942) (xy 28.956 43.942))
+  (wire (pts (xy 40.894 43.942) (xy 42.926 43.942))
     (stroke (width 0) (type default))
   )
@@
     (stroke (width 0) (type default))
   )
-  (wire (pts (xy 39.116 46.482) (xy 26.924 46.482))
+  (wire (pts (xy 53.086 46.482) (xy 40.894 46.482))
     (stroke (width 0) (type default))
   )
@@
     (stroke (width 0) (type default))
   )
-  (wire (pts (xy 28.956 43.942) (xy 28.956 49.022))
+  (wire (pts (xy 42.926 43.942) (xy 42.926 49.022))
     (stroke (width 0) (type default))
   )
@@
     (stroke (width 0) (type default))
   )
-  (wire (pts (xy 28.956 49.022) (xy 28.956 50.8))
+  (wire (pts (xy 42.926 49.022) (xy 42.926 50.8))
     (stroke (width 0) (type default))
   )
@@
     (stroke (width 0) (type default))
   )
+  (wire (pts (xy 100.076 109.982) (xy 110.744 109.982))
+    (stroke (width 0) (type default))
+  )
   (wire (pts (xy 105.41 75.946) (xy 105.41 79.248))
     (stroke (width 0) (type default))
@@
     (stroke (width 0) (type default))
   )
-  (wire (pts (xy 26.924 49.022) (xy 28.956 49.022))
+  (wire (pts (xy 40.894 49.022) (xy 42.926 49.022))
+    (stroke (width 0) (type default))
+  )
+  (wire (pts (xy 100.076 106.934) (xy 110.744 106.934))
     (stroke (width 0) (type default))
   )
@@
     )
   )
-  (symbol (lib_id "Connector_Generic:Conn_01x03") (at 21.844 46.482 180) (unit 1)
-    (in_bom yes) (on_board yes) (dnp no) (fields_autoplaced)
-    (property "Reference" "J2" (at 21.844 38.1 0)
-      (effects (font (size 1.27 1.27)))
-    )
-    (property "Value" "24V In" (at 21.844 40.64 0)
-      (effects (font (size 1.27 1.27)))
-    )
-    (property "Footprint" "" (at 21.844 46.482 0)
-      (effects (font (size 1.27 1.27)) hide)
-    )
-    (property "Datasheet" "~" (at 21.844 46.482 0)
+  (symbol (lib_id "Connector_Generic:Conn_01x03") (at 35.814 46.482 180) (unit 1)
+    (in_bom yes) (on_board yes) (dnp no) (fields_autoplaced)
+    (property "Reference" "J2" (at 35.814 38.1 0)
+      (effects (font (size 1.27 1.27)))
+    )
+    (property "Value" "24V In" (at 35.814 40.64 0)
+      (effects (font (size 1.27 1.27)))
+    )
+    (property "Footprint" "" (at 35.814 46.482 0)
+      (effects (font (size 1.27 1.27)) hide)
+    )
+    (property "Datasheet" "~" (at 35.814 46.482 0)
       (effects (font (size 1.27 1.27)) hide)
     )
@@
     )
   )
-  (symbol (lib_id "power:GND") (at 28.956 50.8 0) (unit 1)
-    (in_bom yes) (on_board yes) (dnp no) (fields_autoplaced)
-    (property "Reference" "#PWR03" (at 28.956 57.15 0)
-      (effects (font (size 1.27 1.27)) hide)
-    )
-    (property "Value" "GND" (at 28.956 55.88 0)
-      (effects (font (size 1.27 1.27)))
-    )
-    (property "Footprint" "" (at 28.956 50.8 0)
-      (effects (font (size 1.27 1.27)) hide)
-    )
-    (property "Datasheet" "" (at 28.956 50.8 0)
+  (symbol (lib_id "power:GND") (at 42.926 50.8 0) (unit 1)
+    (in_bom yes) (on_board yes) (dnp no) (fields_autoplaced)
+    (property "Reference" "#PWR03" (at 42.926 57.15 0)
+      (effects (font (size 1.27 1.27)) hide)
+    )
+    (property "Value" "GND" (at 42.926 55.88 0)
+      (effects (font (size 1.27 1.27)))
+    )
+    (property "Footprint" "" (at 42.926 50.8 0)
+      (effects (font (size 1.27 1.27)) hide)
+    )
+    (property "Datasheet" "" (at 42.926 50.8 0)
       (effects (font (size 1.27 1.27)) hide)
     )
@@
     )
   )
-  (sheet (at 195.834 85.344) (size 39.624 21.59) (fields_autoplaced)
+  (sheet (at 195.834 93.726) (size 24.384 13.208) (fields_autoplaced)
     (stroke (width 0.1524) (type solid))
     (fill (color 0 0 0 0.0000))
-    (property "Sheetname" "CAN" (at 195.834 84.6324 0)
+    (property "Sheetname" "CAN" (at 195.834 93.0144 0)
       (effects (font (size 1.27 1.27)) (justify left bottom))
     )
@@
       (effects (font (size 1.27 1.27)) (justify right))
     )
+    (pin "Fan_Tach" input (at 110.744 106.934 180)
+      (effects (font (size 1.27 1.27)) (justify left))
+    )
+    (pin "Fan_PWM" output (at 110.744 109.982 180)
+      (effects (font (size 1.27 1.27)) (justify left))
+    )
     (instances
       (project "LogicBoard_v1"
@@
     )
   )
-  (sheet (at 39.116 41.148) (size 50.8 27.94) (fields_autoplaced)
+  (sheet (at 74.93 103.886) (size 25.146 8.636) (fields_autoplaced)
     (stroke (width 0.1524) (type solid))
     (fill (color 0 0 0 0.0000))
-    (property "Sheetname" "Power" (at 39.116 40.4364 0)
+    (property "Sheetname" "Fans" (at 74.93 103.1744 0)
       (effects (font (size 1.27 1.27)) (justify left bottom))
     )
-    (property "Sheetfile" "LogicBoard_v1_Power.kicad_sch" (at 39.116 69.6726 0)
+    (property "Sheetfile" "LogicBoard_v1_Fans.kicad_sch" (at 74.93 113.1066 0)
       (effects (font (size 1.27 1.27)) (justify left top))
     )
+    (pin "Fan_Tach" output (at 100.076 106.934 0)
+      (effects (font (size 1.27 1.27)) (justify right))
+    )
+    (pin "Fan_PWM" input (at 100.076 109.982 0)
+      (effects (font (size 1.27 1.27)) (justify right))
+    )
+    (instances
+      (project "LogicBoard_v1"
+        (path "/1e1b062d-fad0-427c-a622-c5b8a80b5268" (page "5"))
+      )
+    )
+  )
+  (sheet (at 53.086 41.148) (size 36.83 18.796) (fields_autoplaced)
+    (stroke (width 0.1524) (type solid))
+    (fill (color 0 0 0 0.0000))
+    (property "Sheetname" "Power" (at 53.086 40.4364 0)
+      (effects (font (size 1.27 1.27)) (justify left bottom))
+    )
+    (property "Sheetfile" "LogicBoard_v1_Power.kicad_sch" (at 53.086 60.5286 0)
+      (effects (font (size 1.27 1.27)) (justify left top))
+    )
     (pin "24V_Protected" output (at 89.916 46.228 0)
       (effects (font (size 1.27 1.27)) (justify right))
@@
       (effects (font (size 1.27 1.27)) (justify right))
     )
-    (pin "24V_Unprotected" input (at 39.116 46.482 180)
-      (effects (font (size 1.27 1.27)) (justify left))
-    )
+    (pin "24V_Unprotected" input (at 53.086 46.482 180)
+      (effects (font (size 1.27 1.27)) (justify left))
+    )

Commit message: Started logic board
Parts:
- added J3: ADC, Connector_Molex:Molex_Micro-Fit_3.0_43650-0500_1x05_P3.00mm_Horizontal, symbol Connector_Generic:Conn_01x05
- added TP1: Duty PWM, TestPoint:TestPoint_THTPad_D1.5mm_Drill0.7mm, symbol Connector:TestPoint
- J1: renamed from J2; footprint (none) -> Connector_Molex:Molex_Micro-Fit_3.0_43650-0300_1x03_P3.00mm_Horizontal; MPN (none) -> 436500300
- J2: renamed from J3; footprint (none) -> Connector_Molex:Molex_Micro-Fit_3.0_43650-0600_1x06_P3.00mm_Horizontal; MPN (none) -> 436500600
- J4: footprint (none) -> Connector_Molex:Molex_Micro-Fit_3.0_43650-0400_1x04_P3.00mm_Horizontal; MPN (none) -> 436500400
Connections:
- net MCU/CS_1: now also J2.5 (Pin_5); no longer J2.2 (Pin_2)
- net MCU/CS_2: now also J2.6 (Pin_6); no longer J2.3 (Pin_3)
- net MCU/MISO: now also J2.2 (Pin_2); no longer J2.4 (Pin_4)
- net MCU/MOSI: now also J2.3 (Pin_3); no longer J2.5 (Pin_5)
- net MCU/PWM: now also TP1.1
- net MCU/SCLK: now also J2.4 (Pin_4); no longer J2.6 (Pin_6)
- net MCU/Temp_Sens renamed MCU/Temp_Sens_SPI
- new net MCU/ADC_1: J3.2 (Pin_2)
- new net MCU/ADC_2: J3.3 (Pin_3)
- new net MCU/ADC_3: J3.4 (Pin_4)
- new net MCU/ADC_4: J3.5 (Pin_5)
- new net MCU/Temp_Sens_ADC: J3.1 (Pin_1)
- no-connect marks 0 -> 3
Other:
- sheet MCU ports: added ADC_1, ADC_2, ADC_3, ADC_4, Temp_Sens_ADC, Temp_Sens_SPI; removed P0_16, P0_21, P0_4, Temp_Sens
- title: Template -> MPPT Logic Board
- moved on the sheet: J4

Commit message: Finsihed logic board
Parts:
- added H1, H2: MountingHole, MountingHole:MountingHole_3.2mm_M3, symbol Mechanical:MountingHole
Changed lines of the file:
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@@
+    )
+  )
+  (symbol (lib_id "Mechanical:MountingHole") (at 235.458 37.338 0) (unit 1)
+    (in_bom yes) (on_board yes) (dnp no) (fields_autoplaced)
+    (property "Reference" "H1" (at 238.76 36.068 0)
+      (effects (font (size 1.27 1.27)) (justify left))
+    )
+    (property "Value" "MountingHole" (at 238.76 38.608 0)
+      (effects (font (size 1.27 1.27)) (justify left))
+    )
+    (property "Footprint" "MountingHole:MountingHole_3.2mm_M3" (at 235.458 37.338 0)
+      (effects (font (size 1.27 1.27)) hide)
+    )
+    (property "Datasheet" "~" (at 235.458 37.338 0)
+      (effects (font (size 1.27 1.27)) hide)
+    )
+    (instances
+      (project "LogicBoard_v1"
+        (path "/1e1b062d-fad0-427c-a622-c5b8a80b5268"
+          (reference "H1") (unit 1)
+        )
+      )
+    )
+  )
+  (symbol (lib_id "Mechanical:MountingHole") (at 235.458 42.672 0) (unit 1)
+    (in_bom yes) (on_board yes) (dnp no) (fields_autoplaced)
+    (property "Reference" "H2" (at 238.76 41.402 0)
+      (effects (font (size 1.27 1.27)) (justify left))
+    )
+    (property "Value" "MountingHole" (at 238.76 43.942 0)
+      (effects (font (size 1.27 1.27)) (justify left))
+    )
+    (property "Footprint" "MountingHole:MountingHole_3.2mm_M3" (at 235.458 42.672 0)
+      (effects (font (size 1.27 1.27)) hide)
+    )
+    (property "Datasheet" "~" (at 235.458 42.672 0)
+      (effects (font (size 1.27 1.27)) hide)
+    )
+    (instances
+      (project "LogicBoard_v1"
+        (path "/1e1b062d-fad0-427c-a622-c5b8a80b5268"
+          (reference "H2") (unit 1)
+        )
+      )
     )
   )
